File: esp-pmsa/esp-pmsa.kicad_pcb (KiCad board)
At the start: 2 copper layers, 40 x 50 mm, 16 parts, among them M1 PMSA003, U1 D1 Mini, U2 BME68x, U3 OPT3001DNPT

Commit message: add gnd zones
Parts:
- moved C1 43.8 mm to (156.6, 114.8), turned to 180 degrees
- moved C2 43.8 mm to (156.6, 113.2), turned to 0 degrees
- moved R2 13.1 mm to (182.5, 83.2), turned to 0 degrees
- moved R1 12.2 mm to (182.5, 81.8), turned to 0 degrees
Routing:
- added copper zone on B.Cu, net GND
- added copper zone on F.Cu, net GND
Changed lines of the file:
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@@
     (user_trace_width 0.762)
     (trace_clearance 0.127)
-    (zone_clearance 0.508)
-    (zone_45_only no)
+    (zone_clearance 0.154)
+    (zone_45_only yes)
     (trace_min 0.127)
     (via_size 0.6)
@@
   )
   (module Resistor_SMD:R_0402_1005Metric (layer Front)
-    (at 174.75 93.75 180)
+    (at 182.5 83.25)
     (descr "Resistor SMD 0402 (1005 Metric), square (rectangular) end terminal, IPC_7351 nominal, (Body size source: IPC-SM-782 page 72, https://www.pcb-3d.com/wordpress/wp-content/uploads/ipc-sm-782a_amendment_1_and_2.pdf), generated with kicad-footprint-generator")
     (tags resistor)
@@
       (effects (font (size 0.6 0.6) (thickness 0.1)))
     )
-    (pad 2 smd roundrect (at 0.51 0 180) (size 0.54 0.64) (layers Front F.Paste F.Mask) (roundrect_rratio 0.25)
+    (pad 2 smd roundrect (at 0.51 0) (size 0.54 0.64) (layers Front F.Paste F.Mask) (roundrect_rratio 0.25)
       (net 13 +3V3))
-    (pad 1 smd roundrect (at -0.51 0 180) (size 0.54 0.64) (layers Front F.Paste F.Mask) (roundrect_rratio 0.25)
+    (pad 1 smd roundrect (at -0.51 0) (size 0.54 0.64) (layers Front F.Paste F.Mask) (roundrect_rratio 0.25)
       (net 9 /SDA))
     (model ${KISYS3DMOD}/Resistor_SMD.3dshapes/R_0402_1005Metric.wrl
@@
   )
   (module Resistor_SMD:R_0402_1005Metric (layer Front)
-    (at 174.75 91.2 180)
+    (at 182.5 81.75)
     (descr "Resistor SMD 0402 (1005 Metric), square (rectangular) end terminal, IPC_7351 nominal, (Body size source: IPC-SM-782 page 72, https://www.pcb-3d.com/wordpress/wp-content/uploads/ipc-sm-782a_amendment_1_and_2.pdf), generated with kicad-footprint-generator")
     (tags resistor)
@@
       (effects (font (size 0.6 0.6) (thickness 0.1)))
     )
-    (pad 2 smd roundrect (at 0.51 0 180) (size 0.54 0.64) (layers Front F.Paste F.Mask) (roundrect_rratio 0.25)
+    (pad 2 smd roundrect (at 0.51 0) (size 0.54 0.64) (layers Front F.Paste F.Mask) (roundrect_rratio 0.25)
       (net 13 +3V3))
-    (pad 1 smd roundrect (at -0.51 0 180) (size 0.54 0.64) (layers Front F.Paste F.Mask) (roundrect_rratio 0.25)
+    (pad 1 smd roundrect (at -0.51 0) (size 0.54 0.64) (layers Front F.Paste F.Mask) (roundrect_rratio 0.25)
       (net 8 /SCL))
     (model ${KISYS3DMOD}/Resistor_SMD.3dshapes/R_0402_1005Metric.wrl
@@
   )
   (module Capacitor_SMD:C_0603_1608Metric_Pad1.05x0.95mm_HandSolder (layer Front)
-    (at 188.25 82.975 270)
+    (at 156.575 113.25)
     (descr "Capacitor SMD 0603 (1608 Metric), square (rectangular) end terminal, IPC_7351 nominal with elongated pad for handsoldering. (Body size source: http://www.tortai-tech.com/upload/download/2011102023233369053.pdf), generated with kicad-footprint-generator")
     (tags "capacitor handsolder")
     (attr smd)
-    (fp_text reference C2 (at 2.5 0 90) (layer F.SilkS)
-      (effects (font (size 0.8 0.8) (thickness 0.1524)))
-    )
-    (fp_text value 10uF (at 0 1.43 90) (layer F.Fab)
+    (fp_text reference C2 (at 2.5 0) (layer F.SilkS)
+      (effects (font (size 0.8 0.8) (thickness 0.1524)))
+    )
+    (fp_text value 10uF (at 0 1.43) (layer F.Fab)
       (effects (font (size 0.6 0.6) (thickness 0.1)))
     )
@@
     (fp_line (start -0.8 -0.4) (end 0.8 -0.4) (layer F.Fab) (width 0.1))
     (fp_line (start -0.8 0.4) (end -0.8 -0.4) (layer F.Fab) (width 0.1))
-    (fp_text user %R (at 0 0 90) (layer F.Fab)
-      (effects (font (size 0.6 0.6) (thickness 0.1)))
-    )
-    (pad 2 smd roundrect (at 0.875 0 270) (size 1.05 0.95) (layers Front F.Paste F.Mask) (roundrect_rratio 0.25)
-      (net 2 GND))
-    (pad 1 smd roundrect (at -0.875 0 270) (size 1.05 0.95) (layers Front F.Paste F.Mask) (roundrect_rratio 0.25)
+    (fp_text user %R (at 0 0) (layer F.Fab)
+      (effects (font (size 0.6 0.6) (thickness 0.1)))
+    )
+    (pad 2 smd roundrect (at 0.875 0) (size 1.05 0.95) (layers Front F.Paste F.Mask) (roundrect_rratio 0.25)
+      (net 2 GND))
+    (pad 1 smd roundrect (at -0.875 0) (size 1.05 0.95) (layers Front F.Paste F.Mask) (roundrect_rratio 0.25)
       (net 1 +5V))
     (model ${KISYS3DMOD}/Capacitor_SMD.3dshapes/C_0603_1608Metric.wrl
@@
   )
   (module Capacitor_SMD:C_0603_1608Metric_Pad1.05x0.95mm_HandSolder (layer Front)
-    (at 186.75 82.975 90)
+    (at 156.575 114.75 180)
     (descr "Capacitor SMD 0603 (1608 Metric), square (rectangular) end terminal, IPC_7351 nominal with elongated pad for handsoldering. (Body size source: http://www.tortai-tech.com/upload/download/2011102023233369053.pdf), generated with kicad-footprint-generator")
     (tags "capacitor handsolder")
     (attr smd)
-    (fp_text reference C1 (at -2.5 0 90) (layer F.SilkS)
-      (effects (font (size 0.8 0.8) (thickness 0.1524)))
-    )
-    (fp_text value 10uF (at 0 1.43 90) (layer F.Fab)
+    (fp_text reference C1 (at -2.5 0) (layer F.SilkS)
+      (effects (font (size 0.8 0.8) (thickness 0.1524)))
+    )
+    (fp_text value 10uF (at 0 1.43) (layer F.Fab)
       (effects (font (size 0.6 0.6) (thickness 0.1)))
     )
@@
     (fp_line (start -0.8 -0.4) (end 0.8 -0.4) (layer F.Fab) (width 0.1))
     (fp_line (start -0.8 0.4) (end -0.8 -0.4) (layer F.Fab) (width 0.1))
-    (fp_text user %R (at 0 0 90) (layer F.Fab)
-      (effects (font (size 0.6 0.6) (thickness 0.1)))
-    )
-    (pad 2 smd roundrect (at 0.875 0 90) (size 1.05 0.95) (layers Front F.Paste F.Mask) (roundrect_rratio 0.25)
+    (fp_text user %R (at 0 0) (layer F.Fab)
+      (effects (font (size 0.6 0.6) (thickness 0.1)))
+    )
+    (pad 2 smd roundrect (at 0.875 0 180) (size 1.05 0.95) (layers Front F.Paste F.Mask) (roundrect_rratio 0.25)
       (net 1 +5V))
-    (pad 1 smd roundrect (at -0.875 0 90) (size 1.05 0.95) (layers Front F.Paste F.Mask) (roundrect_rratio 0.25)
+    (pad 1 smd roundrect (at -0.875 0 180) (size 1.05 0.95) (layers Front F.Paste F.Mask) (roundrect_rratio 0.25)
       (net 2 GND))
     (model ${KISYS3DMOD}/Capacitor_SMD.3dshapes/C_0603_1608Metric.wrl
@@
   (gr_line (start 150 122.5) (end 150 77.5) (layer Edge.Cuts) (width 0.05))
   (gr_line (start 182.5 80) (end 157.5 80) (layer Edge.Cuts) (width 0.05))
+  (zone (net 2) (net_name GND) (layer Front) (hatch edge 0.508)
+    (connect_pads (clearance 0.154))
+    (min_thickness 0.154)
+    (fill yes (arc_segments 32) (thermal_gap 0.254) (thermal_bridge_width 0.254) (smoothing fillet) (radius 0.075))
+    (polygon
+      (pts
+        (xy 190 125) (xy 150 125) (xy 150 75) (xy 190 75)
+      )
+    )
+  )
+  (zone (net 2) (net_name GND) (layer Back) (hatch edge 0.508)
+    (connect_pads (clearance 0.154))
+    (min_thickness 0.154)
+    (fill yes (arc_segments 32) (thermal_gap 0.254) (thermal_bridge_width 0.254) (smoothing fillet) (radius 0.075))
+    (polygon
+      (pts
+        (xy 190 125) (xy 150 125) (xy 150 75) (xy 190 75)
+      )
+    )
+  )
 )

Commit message: ok this is silly
Parts:
- added C7: 10uF, Capacitor_SMD:C_0603_1608Metric_Pad1.05x0.95mm_HandSolder, F.Cu at (153.0, 109.9)
- added C8: 10uF, Capacitor_SMD:C_0603_1608Metric_Pad1.05x0.95mm_HandSolder, F.Cu at (153.0, 108.2)
- added C9: 100nF, Capacitor_SMD:C_0402_1005Metric, F.Cu at (152.0, 90.0)
- added J1: USB_B_Micro, 41-EasyEDA-Edits:MICRO-USB-SMD_U254-051T-4BH83-F1S_C397452, F.Cu at (177.8, 116.2)
- added J2: ESP-PROG, 11-My-Edits:TC2030_IDCBox_2x03_P1.25mm_Vertical_3D, F.Cu at (199.9, 106.2)
- added SW1: ~RESET, 41-EasyEDA-Edits:KEY-SMD_4P-SKSCLXX010, F.Cu at (151.8, 93.8)
- added SW2: ~BOOT, 41-EasyEDA-Edits:KEY-SMD_4P-SKSCLXX010, F.Cu at (151.8, 100.0)
- added U4: XC6220B331MR, Package_TO_SOT_SMD:SOT-23-5, F.Cu at (169.0, 109.5)
- C1, C2: footprint Capacitor_SMD:C_0603_1608Metric_Pad1.05x0.95mm_HandSolder -> Capacitor_SMD:C_0402_1005Metric
- C3, C4: moved to F.Cu
- U1: value D1 Mini -> ESP32-C3-WROOM-02; footprint 11-My-Edits:WEMOS_D1_mini_SMT -> 10-My-Footprints:ESP32-C3-WROOM-02-PTHPad
- moved R1 24.8 mm to (158.4, 87.5), turned to 180 degrees
- moved R2 24.3 mm to (158.4, 86.0), turned to 180 degrees
- moved C1 15.6 mm to (171.5, 110.1), turned to 270 degrees
- moved C3 14.0 mm to (161.4, 114.1), turned to 0 degrees
- moved C2 13.9 mm to (169.0, 107.0)
- moved U1 8.62 mm to (170.0, 89.2), turned to 0 degrees
- moved C5 7.11 mm to (170.1, 114.1), turned to 180 degrees
- moved C4 6.17 mm to (161.4, 115.4), turned to 180 degrees
- moved C6 6.03 mm to (170.1, 115.4), turned to 180 degrees
- moved U2 4.28 mm to (165.8, 122.0)
- moved U3 4.28 mm to (165.8, 122.0)
- moved M1 1.25 mm to (170.0, 97.5)
Connections:
- C2 pad 1: +5V -> +3V3
- C3 pad 1: /VCC_SENS -> /VCC_BME
- C4 pad 2: /VCC_SENS -> /VCC_BME
- C5 pad 1: /VCC_SENS -> /VCC_ALS
- C6 pad 1: /VCC_SENS -> /VCC_ALS
- M1 pad 7: /U0TX_B -> /PMS_RX
- M1 pad 9: /U0RX_B -> /PMS_TX
- U1 pad 1: /~WAKE -> +3V3
- U1 pad 10: GND -> /RGB
- U1 pad 11: Net-(U1-Pad11) -> /U0RXD
- U1 pad 12: /~PMS_SET -> /U0TXD
- U1 pad 13: /SDA -> /USB_D-
- U1 pad 14: /SCL -> /USB_D+
- U1 pad 15: Net-(U1-Pad15) -> /~PMS_RST
- U1 pad 16: Net-(U1-Pad16) -> /~PMS_SET
- U1 pad 2: Net-(U1-Pad2) -> /~RST
- U1 pad 3: /~WAKE -> /SDA
- U1 pad 4: /RGB -> /SCL
- U1 pad 5: /VCC_SENS -> /VCC_ALS
- U1 pad 6: /U0RX_B -> /VCC_BME
- U1 pad 7: /U0TX_B -> Net-(U1-Pad7)
- U1 pad 8: +5V -> /~BOOT
- U1 pad 9: +3V3 -> GND
- U2 pad 2: /VCC_SENS -> /VCC_BME
- U2 pad 6: /VCC_SENS -> /VCC_BME
- U2 pad 8: /VCC_SENS -> /VCC_BME
- U3 pad 1: /VCC_SENS -> /VCC_ALS
Routing:
- net /~RST: track 0.00 -> 5.96 mm
- net GND: track 0.00 -> 1.90 mm
- net /VCC_BME: track 0.00 -> 1.25 mm
- net /VCC_ALS: track 0.00 -> 1.25 mm
- added copper zone on F.Cu, net +5V
Other:
- outline, holes or cut-outs redrawn

Commit message: KISS
Parts:
- removed C1, C2: 10uF, Capacitor_SMD:C_0402_1005Metric
- removed C5: 1uF, Capacitor_SMD:C_0402_1005Metric
- removed C6, C9: 100nF, Capacitor_SMD:C_0402_1005Metric
- removed J1: USB_B_Micro, 41-EasyEDA-Edits:MICRO-USB-SMD_U254-051T-4BH83-F1S_C397452
- removed J2: ESP-PROG, 11-My-Edits:TC2030_IDCBox_2x03_P1.25mm_Vertical_3D
- removed R1, R2: 4K7, Resistor_SMD:R_0402_1005Metric
- removed SW1: ~RESET, 41-EasyEDA-Edits:KEY-SMD_4P-SKSCLXX010
- removed SW2: ~BOOT, 41-EasyEDA-Edits:KEY-SMD_4P-SKSCLXX010
- removed U4: XC6220B331MR, Package_TO_SOT_SMD:SOT-23-5
- U1: value ESP32-C3-WROOM-02 -> WeMos_D1_mini_Labels; footprint 10-My-Footprints:ESP32-C3-WROOM-02-PTHPad -> 11-My-Edits:WEMOS_D1_mini
- moved U3 34.9 mm to (186.2, 93.8)
- moved C3 19.9 mm to (181.3, 115.3)
- moved C4 19.9 mm to (181.3, 116.5)
- moved U1 7.00 mm to (170.0, 96.2)
- moved U2 4.25 mm to (170.0, 122.0)
Connections:
- C3 pad 1: /VCC_BME -> /VCC_SENS
- C4 pad 2: /VCC_BME -> /VCC_SENS
- M1 pad 8: Net-(M1-Pad6) -> Net-(M1-Pad8)
- U1 pad 1: +3V3 -> /~WAKE
- U1 pad 10: /RGB -> GND
- U1 pad 11: /U0RXD -> Net-(U1-Pad11)
- U1 pad 12: /U0TXD -> /VCC_SENS
- U1 pad 13: /USB_D- -> /SDA
- U1 pad 14: /USB_D+ -> /SCL
- U1 pad 15: /~PMS_RST -> /U0RXD
- U1 pad 16: /~PMS_SET -> /U0TXD
- U1 pad 2: /~RST -> Net-(U1-Pad2)
- U1 pad 3: /SDA -> /~WAKE
- U1 pad 4: /SCL -> /~PMS_RST
- U1 pad 5: /VCC_ALS -> /~PMS_SET
- U1 pad 6: /VCC_BME -> /PMS_TX
- U1 pad 7: Net-(U1-Pad7) -> /PMS_RX
- U1 pad 8: /~BOOT -> +3V3
- U1 pad 9: GND -> +5V
- U2 pad 2: /VCC_BME -> /VCC_SENS
- U2 pad 6: /VCC_BME -> /VCC_SENS
- U2 pad 8: /VCC_BME -> /VCC_SENS
- U3 pad 1: /VCC_ALS -> /VCC_SENS
Routing:
- net /VCC_SENS: track 0.00 -> 46.4 mm, vias 0 -> 1
- net /SCL: track 0.00 -> 38.2 mm
- net /SDA: track 0.00 -> 36.3 mm
- net /PMS_RX: track 0.00 -> 16.2 mm, vias 0 -> 1
- net /PMS_TX: track 0.00 -> 12.3 mm
- net /~RST: track 5.96 -> 0.00 mm
- net GND: track 1.90 -> 3.89 mm, vias 0 -> 2
- net /VCC_BME: track 1.25 -> 0.00 mm
- net /VCC_ALS: track 1.25 -> 0.00 mm
Other:
- outline, holes or cut-outs redrawn

Commit message: still don't like
Routing:
- net /PMS_RX: track 16.2 -> 0.00 mm, vias 1 -> 0
- net /PMS_TX: track 12.3 -> 0.00 mm
- net /VCC_SENS: track 46.4 -> 41.1 mm, vias 1 -> 0
- net GND: track 3.89 -> 0.00 mm, vias 2 -> 0
- net /SDA: track 36.3 -> 35.4 mm

Commit message: v0.1
Parts:
- moved C3 12.5 mm to (169.2, 119.0), turned to 90 degrees
- moved C4 10.8 mm to (170.8, 119.0), turned to 270 degrees
- moved H2 2.50 mm to (187.5, 120.0)
- moved H4 2.50 mm to (152.5, 120.0)
- moved U2 2.50 mm to (170.0, 119.5)
- moved C7 0.28 mm to (153.2, 109.8)
- moved C8 0.28 mm to (153.2, 108.3)
- moved U1 0.25 mm to (170.0, 96.0)
- moved U3 0.25 mm to (186.2, 93.5)
Routing:
- net +5V: track 0.00 -> 39.4 mm
- net /~PMS_RST: track 0.00 -> 23.1 mm
- net /PMS_RX: track 0.00 -> 17.0 mm, vias 0 -> 1
- net /~PMS_SET: track 0.00 -> 14.8 mm
- net /PMS_TX: track 0.00 -> 13.5 mm
- net /~WAKE: track 0.00 -> 7.79 mm
- net /SCL: track 38.2 -> 35.5 mm
- net /VCC_SENS: track 41.1 -> 42.8 mm, vias 0 -> 1
- net /SDA: track 35.4 -> 33.8 mm
- net GND: vias 0 -> 25
- removed copper zone on F.Cu, net +5V
Other:
- board size 40 x 50 mm -> 40 x 47.5 mm
- board text added: "vriska did nothing wrong"
