File: esp-pmsa/esp-pmsa.sch (KiCad schematic (older format))
At the start: 16 parts, among them M1 PMSA003, U1 D1 Mini, U2 BME68x, U3 OPT3001DNPT

Commit message: ok this is silly
Parts:
- removed U1: D1 Mini, 11-My-Edits:WEMOS_D1_mini_SMT, symbol 1_My_Symbols:WeMos_D1_mini_Labels
- added C7, C8: 10uF, Capacitor_SMD:C_0603_1608Metric_Pad1.05x0.95mm_HandSolder, symbol Device:C_Small
- added C9: 100nF, Capacitor_SMD:C_0402_1005Metric, symbol Device:C_Small
- added J1: USB_B_Micro, 41-EasyEDA-Edits:MICRO-USB-SMD_U254-051T-4BH83-F1S_C397452, symbol Connector:USB_B_Micro
- added J2: ESP-PROG, 11-My-Edits:TC2030_IDCBox_2x03_P1.25mm_Vertical_3D, symbol Connector_Generic:Conn_02x03_Odd_Even
- added SW1: ~RESET, 41-EasyEDA-Edits:KEY-SMD_4P-SKSCLXX010, symbol Switch:SW_Push
- added SW2: ~BOOT, 41-EasyEDA-Edits:KEY-SMD_4P-SKSCLXX010, symbol Switch:SW_Push
- added U1: ESP32-C3-WROOM-02, 10-My-Footprints:ESP32-C3-WROOM-02-PTHPad, symbol 1_My_Symbols:ESP32-C3-WROOM-02-8266Style
- added U4: XC6220B331MR, Package_TO_SOT_SMD:SOT-23-5, symbol Regulator_Linear:XC6220B331MR
- C1, C2: footprint Capacitor_SMD:C_0603_1608Metric_Pad1.05x0.95mm_HandSolder -> Capacitor_SMD:C_0402_1005Metric; LCSC C19702 -> C15525; MPN CL10A106KP8NNNC -> CL05A106MQ5NUNC
Connections:
- net labels added: PMS_RX, PMS_TX, U0RXD, U0TXD, USB_D+, USB_D-, USB_ID, VCC_ALS, VCC_BME, VPP, ~BOOT, ~RST
- net labels removed: U0RX_B, U0TX_B, VCC_SENS, ~WAKE
- wire segments 96 -> 140
- no-connect marks 5 -> 4
Other:
- moved on the sheet: C1, C2, C3, C4, C5, C6, H1, H2, H3, H4, M1, R1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

Commit message: tweak
Parts:
- M1: symbol 1_My_Symbols:PMSA003 -> esp-pmsa-rescue:PMSA003-1_My_Symbols
Changed lines of the file:
@@
 	6000 3750 6000 3850
 $Comp
-L 1_My_Symbols:PMSA003 M1
+L esp-pmsa-rescue:PMSA003-1_My_Symbols M1
 U 1 1 6071E0E3
 P 9000 2750
