File: esp-pmsa/esp-pmsa.sch (KiCad schematic (older format))
At the start: 24 parts, among them J1 USB_B_Micro, J2 ESP-PROG, M1 PMSA003, SW1 ~RESET, SW2 ~BOOT, U1 ESP32-C3-WROOM-02, U2 BME68x, U3 OPT3001DNPT, U4 XC6220B331MR

Commit message: KISS
Parts:
- removed C1, C2: 10uF, Capacitor_SMD:C_0402_1005Metric, symbol Device:C_Small
- removed C5: 1uF, Capacitor_SMD:C_0402_1005Metric, symbol Device:C_Small
- removed C6, C9: 100nF, Capacitor_SMD:C_0402_1005Metric, symbol Device:C_Small
- removed J1: USB_B_Micro, 41-EasyEDA-Edits:MICRO-USB-SMD_U254-051T-4BH83-F1S_C397452, symbol Connector:USB_B_Micro
- removed J2: ESP-PROG, 11-My-Edits:TC2030_IDCBox_2x03_P1.25mm_Vertical_3D, symbol Connector_Generic:Conn_02x03_Odd_Even
- removed SW1: ~RESET, 41-EasyEDA-Edits:KEY-SMD_4P-SKSCLXX010, symbol Switch:SW_Push
- removed SW2: ~BOOT, 41-EasyEDA-Edits:KEY-SMD_4P-SKSCLXX010, symbol Switch:SW_Push
- removed U1: ESP32-C3-WROOM-02, 10-My-Footprints:ESP32-C3-WROOM-02-PTHPad, symbol 1_My_Symbols:ESP32-C3-WROOM-02-8266Style
- removed U4: XC6220B331MR, Package_TO_SOT_SMD:SOT-23-5, symbol Regulator_Linear:XC6220B331MR
- added U1: WeMos_D1_mini_Labels, 11-My-Edits:WEMOS_D1_mini, symbol 1_My_Symbols:WeMos_D1_mini_Labels
Connections:
- net labels added: VCC_SENS, ~WAKE
- net labels removed: RGB, USB_D+, USB_D-, USB_ID, VCC_ALS, VCC_BME, VPP, ~BOOT, ~RST
- wire segments 140 -> 85
Other:
- moved on the sheet: C3, C4, C7, C8, H1, H2, H3, H4, M1, R1, R2, U2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

Commit message: switch to ESP-C3-F
Parts:
- removed U1: WeMos_D1_mini_Labels, 11-My-Edits:WEMOS_D1_mini, symbol 1_My_Symbols:WeMos_D1_mini_Labels
- added C1, C2: 10u, Capacitor_SMD:C_0402_1005Metric, symbol Device:C_Small
- added C5: 1u, Capacitor_SMD:C_0402_1005Metric, symbol Device:C_Small
- added C6, C9: 0.1u, Capacitor_SMD:C_0402_1005Metric, symbol Device:C_Small
- added D1: APA104-12-3535, 21-SnapEDA-zip:LED_APA104-12-3535, symbol 1_My_Symbols:APA104-12-3535
- added J1: USB_C_Receptacle_USB2.0_304S-ACP16, 41-EasyEDA-Edits:USB-C-SMD_TYPEC-304S-ACP16, symbol 1_My_Symbols:USB_C_Receptacle_USB2.0_304S-ACP16
- added J2: ESP-PROG, 11-My-Edits:TC2030_IDCBox_2x03_P1.25mm_Vertical_3D, symbol Connector_Generic:Conn_02x03_Odd_Even
- added R3, R4: 5k1, Resistor_SMD:R_0402_1005Metric, symbol Device:R_Small
- added SW1: Reset, 41-EasyEDA-Edits:SW-SMD_SKSLLAE010-3D, symbol Switch:SW_Push
- added SW2: Boot, 41-EasyEDA-Edits:SW-SMD_SKSLLAE010-3D, symbol Switch:SW_Push
- added U1: ESP32-C3F, 11-My-Edits:ESP-12H, symbol 1_My_Symbols:ESP32-C3F
- added U4: XC6220B331MR, Package_TO_SOT_SMD:SOT-23-5, symbol Regulator_Linear:XC6220B331MR
- C3: value 1uF -> 1u
- C4: value 100nF -> 0.1u
- C7, C8: value 10uF -> 10u
- M1: symbol 1_My_Symbols:PMSA003 -> esp-pmsa-rescue:PMSA003-1_My_Symbols
- R1, R2: value 4K7 -> 4k7
Connections:
- net +3V3: now also R1.1, R2.1, C2.1, U1.8 (VCC), U4.5 (VOUT)
- net +5V: now also C1.2, D1.4 (VDD), J1.A4B9 (VBUS), J1.B4A9 (VBUS), U4.1 (VIN), U4.3 (CE)
- net GND: now also C4.2, C1.1, C2.2, C5.2, C6.2, C9.1, D1.2 (VSS), J1.A1B12 (GND), J1.B1A12 (GND), J1.S1 (SHIELD), J2.4 (Pin_4), R3.1, R4.1, SW1.1, SW2.1, U1.15 (GND), U4.2 (GND); no longer C4.1
- net PMS_RX: now also U1.1 (IO0)
- net PMS_TX: now also U1.2 (IO1)
- net SCL: now also R1.2, U1.7 (MTDI/IO5); no longer R1.1
- net SDA: now also R2.2, U1.6 (MTMS/IO4); no longer R2.1
- net U0RXD: now also J2.5 (Pin_5), U1.21 (IO20/U0RX)
- net U0TXD: now also J2.3 (Pin_3), U1.22 (IO21/U0TX)
- net ~PMS_RST: now also U1.5 (IO3)
- net ~PMS_SET: now also U1.4 (IO2)
- net at M1.6 (NC): now also M1.8 (NC)
- net VCC_SENS renamed VCC_BME
- net VCC_BME: now also C4.1, U1.13 (MTDO/IO7); no longer C4.2, R1.2, R2.2, U3.1 (VDD)
- new net: U1.10 (NC), U1.11 (NC), U1.14 (NC), U1.9 (NC)
- new net: J1.A5 (CC1), R3.2
- new net: J1.B5 (CC2), R4.2
- new net RGB: D1.3 (DIN), U1.17 (IO10)
- new net USB_D+: J1.A6 (D+), J1.B6 (D+), U1.19 (IO19/D+)
- new net USB_D-: J1.A7 (D-), J1.B7 (D-), U1.20 (IO18/D-)
- new net VCC_ALS: C5.1, C6.1, U1.12 (MTCK/IO6), U3.1 (VDD)
- new net VPP: J2.2 (Pin_2)
- new net ~BOOT: J2.6 (Pin_6), SW2.2, U1.18 (~BOOT~/IO9)
- new net ~RST: C9.2, J2.1 (Pin_1), SW1.2, U1.3 (EN)
- no-connect marks 4 -> 6
Other:
- moved on the sheet: C3, C4, C7, C8, H1, H2, H3, H4, M1, R1, R2, U2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
