File: esp-pmsa/esp-pmsa.sch (KiCad schematic (older format))
At the start: 27 parts, among them J1 USB_C_Receptacle_USB2.0_304S-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, J2 ESP-PROG, M1 PMSA003, SW1 Reset, SW2 Boot, U1 ESP32-C3F, U2 BME68x, U3 OPT3001DNPT, U4 XC6220B331MR

Commit message: okeydokey!
Parts:
- SW1, SW2: symbol Switch:SW_Push -> 1_My_Symbols:SW_Push_MP
- U4: value XC6220B331MR -> XC6210B332MR; symbol Regulator_Linear:XC6220B331MR -> 2_Collected_Symbols:XC6210B332MR; LCSC (none) -> XC6210B332MR-G
Connections:
- net GND: now also SW1.MP, SW2.MP
Other:
- moved on the sheet: C2, C9, U4
Changed lines of the file:
@@
 L power:PWR_FLAG #FLG03
 U 1 1 6070DFE3
-P 2250 4550
-F 0 "#FLG03" H 2250 4625 50  0001 C CNN
-F 1 "PWR_FLAG" V 2250 4677 50  0000 L CNN
-F 2 "" H 2250 4550 50  0001 C CNN
-F 3 "~" H 2250 4550 50  0001 C CNN
-	1    2250 4550
-	0    -1   -1   0
+P 2100 4450
+F 0 "#FLG03" H 2100 4525 50  0001 C CNN
+F 1 "PWR_FLAG" H 2100 4623 50  0000 C CNN
+F 2 "" H 2100 4450 50  0001 C CNN
+F 3 "~" H 2100 4450 50  0001 C CNN
+	1    2100 4450
+	1    0    0    -1
 $EndComp
 $Comp
@@
 L Device:C_Small C2
 U 1 1 60722DA8
-P 3250 4200
-F 0 "C2" H 3365 4246 50  0000 L CNN
-F 1 "10u" H 3365 4155 50  0000 L CNN
-F 2 "Capacitor_SMD:C_0402_1005Metric" H 3288 4050 50  0001 C CNN
-F 3 "~" H 3250 4200 50  0001 C CNN
-F 4 "C15525" H 3250 4200 50  0001 C CNN "LCSC"
-F 5 "CL05A106MQ5NUNC" H 3250 4200 50  0001 C CNN "MPN"
-F 6 "Samsung Electro-Mechanics" H 3250 4200 50  0001 C CNN "Manufacturer"
-	1    3250 4200
+P 3250 4250
+F 0 "C2" H 3365 4296 50  0000 L CNN
+F 1 "10u" H 3365 4205 50  0000 L CNN
+F 2 "Capacitor_SMD:C_0402_1005Metric" H 3288 4100 50  0001 C CNN
+F 3 "~" H 3250 4250 50  0001 C CNN
+F 4 "C15525" H 3250 4250 50  0001 C CNN "LCSC"
+F 5 "CL05A106MQ5NUNC" H 3250 4250 50  0001 C CNN "MPN"
+F 6 "Samsung Electro-Mechanics" H 3250 4250 50  0001 C CNN "Manufacturer"
+	1    3250 4250
 	1    0    0    -1
 $EndComp
@@
 L power:+5V #PWR04
 U 1 1 60705AA7
-P 1750 3650
-F 0 "#PWR04" H 1750 3500 50  0001 C CNN
-F 1 "+5V" H 1765 3823 50  0000 C CNN
-F 2 "" H 1750 3650 50  0001 C CNN
-F 3 "" H 1750 3650 50  0001 C CNN
-	1    1750 3650
+P 1750 3900
+F 0 "#PWR04" H 1750 3750 50  0001 C CNN
+F 1 "+5V" H 1765 4073 50  0000 C CNN
+F 2 "" H 1750 3900 50  0001 C CNN
+F 3 "" H 1750 3900 50  0001 C CNN
+	1    1750 3900
 	-1   0    0    -1
 $EndComp
@@
 VCC_ALS
 $Comp
-L Regulator_Linear:XC6220B331MR U4
+L 2_Collected_Symbols:XC6210B332MR U4
 U 1 1 608399F2
-P 2500 4000
-F 0 "U4" H 2500 4367 50  0000 C CNN
-F 1 "XC6220B331MR" H 2500 4276 50  0000 C CNN
-F 2 "Package_TO_SOT_SMD:SOT-23-5" H 2500 4000 50  0001 C CNN
-F 3 "https://www.torexsemi.com/file/xc6220/XC6220.pdf" H 3250 3000 50  0001 C CNN
-F 4 "0;0;-180" H 2500 4000 50  0001 C CNN "JLCPCB_CORRECTION"
-	1    2500 4000
-	1    0    0    -1
-$EndComp
-Wire Wire Line
-	1750 3900 1950 3900
-Wire Wire Line
-	2500 4400 2500 4450
-Wire Wire Line
-	1750 4450 1750 4300
+P 2500 4100
+F 0 "U4" H 2500 4467 50  0000 C CNN
+F 1 "XC6210B332MR" H 2500 4376 50  0000 C CNN
+F 2 "Package_TO_SOT_SMD:SOT-23-5" H 2500 4100 50  0001 C CNN
+F 3 "https://www.torexsemi.com/file/xc6220/XC6220.pdf" H 3250 3100 50  0001 C CNN
+F 4 "0;0;-180" H 2500 4100 50  0001 C CNN "JLCPCB_CORRECTION"
+F 5 "XC6210B332MR-G" H 2500 4100 50  0001 C CNN "LCSC"
+	1    2500 4100
+	1    0    0    -1
+$EndComp
+Wire Wire Line
+	1750 4000 2050 4000
+Wire Wire Line
+	2500 4350 2500 4500
+Wire Wire Line
+	1750 4500 1750 4300
 $Comp
 L Device:C_Small C7
@@
 L power:GND #PWR011
 U 1 1 60872BA0
-P 2500 4600
-F 0 "#PWR011" H 2500 4350 50  0001 C CNN
-F 1 "GND" H 2505 4427 50  0000 C CNN
-F 2 "" H 2500 4600 50  0001 C CNN
-F 3 "" H 2500 4600 50  0001 C CNN
-	1    2500 4600
-	1    0    0    -1
-$EndComp
-Wire Wire Line
-	2500 4600 2500 4550
-Connection ~ 2500 4450
+P 2500 4550
+F 0 "#PWR011" H 2500 4300 50  0001 C CNN
+F 1 "GND" H 2505 4377 50  0000 C CNN
+F 2 "" H 2500 4550 50  0001 C CNN
+F 3 "" H 2500 4550 50  0001 C CNN
+	1    2500 4550
+	1    0    0    -1
+$EndComp
+Connection ~ 2500 4500
 $Comp
 L Device:C_Small C8
@@
 $EndComp
 Wire Wire Line
-	3250 4300 3250 4450
-Wire Wire Line
-	3250 4450 2500 4450
-Wire Wire Line
-	3000 3900 3250 3900
-Wire Wire Line
-	3250 3900 3250 4100
-Connection ~ 3250 3900
+	3250 4350 3250 4500
+Wire Wire Line
+	3250 4500 2500 4500
+Wire Wire Line
+	2850 4000 3250 4000
+Wire Wire Line
+	3250 4000 3250 4150
+Connection ~ 3250 4000
 $Comp
 L power:+3V3 #PWR05
 U 1 1 60884927
-P 3250 3650
-F 0 "#PWR05" H 3250 3500 50  0001 C CNN
-F 1 "+3V3" H 3250 3800 50  0000 C CNN
-F 2 "" H 3250 3650 50  0001 C CNN
-F 3 "" H 3250 3650 50  0001 C CNN
-	1    3250 3650
+P 3250 3900
+F 0 "#PWR05" H 3250 3750 50  0001 C CNN
+F 1 "+3V3" H 3250 4050 50  0000 C CNN
+F 2 "" H 3250 3900 50  0001 C CNN
+F 3 "" H 3250 3900 50  0001 C CNN
+	1    3250 3900
 	1    0    0    -1
 $EndComp
 NoConn ~ 6650 1650
 $Comp
-L Switch:SW_Push SW2
+L 1_My_Symbols:SW_Push_MP SW2
 U 1 1 607750E9
 P 6250 5750
-F 0 "SW2" V 6296 5702 50  0000 R CNN
-F 1 "Boot" V 6205 5702 50  0000 R CNN
+F 0 "SW2" V 6296 5898 50  0000 L CNN
+F 1 "Boot" V 6205 5898 50  0000 L CNN
 F 2 "41-EasyEDA-Edits:SW-SMD_SKSLLAE010-3D" H 6250 5950 50  0001 C CNN
 F 3 "~" H 6250 5950 50  0001 C CNN
@@
 F 6 "ALPS Alpine" H 6250 5750 50  0001 C CNN "Manufacturer"
 	1    6250 5750
-	0    -1   -1   0
+	0    1    -1   0
 $EndComp
 $Comp
 L Device:C_Small C9
 U 1 1 60775C7C
+P 5000 5750
+F 0 "C9" H 4908 5704 50  0000 R CNN
+F 1 "0.1u" H 4908 5795 50  0000 R CNN
+F 2 "Capacitor_SMD:C_0402_1005Metric" H 5000 5750 50  0001 C CNN
+F 3 "~" H 5000 5750 50  0001 C CNN
+F 4 "C1525" H 5000 5750 50  0001 C CNN "LCSC"
+F 5 "Samsung Electro-Mechanics" H 5000 5750 50  0001 C CNN "Manufacturer"
+F 6 "CL05B104KO5NNNC" H 5000 5750 50  0001 C CNN "MPN"
+	1    5000 5750
+	-1   0    0    1
+$EndComp
+$Comp
+L 1_My_Symbols:SW_Push_MP SW1
+U 1 1 6077308A
 P 5500 5750
-F 0 "C9" H 5591 5704 50  0000 L CNN
-F 1 "0.1u" H 5591 5795 50  0000 L CNN
-F 2 "Capacitor_SMD:C_0402_1005Metric" H 5500 5750 50  0001 C CNN
-F 3 "~" H 5500 5750 50  0001 C CNN
-F 4 "C1525" H 5500 5750 50  0001 C CNN "LCSC"
-F 5 "Samsung Electro-Mechanics" H 5500 5750 50  0001 C CNN "Manufacturer"
-F 6 "CL05B104KO5NNNC" H 5500 5750 50  0001 C CNN "MPN"
+F 0 "SW1" V 5546 5898 50  0000 L CNN
+F 1 "Reset" V 5455 5898 50  0000 L CNN
+F 2 "41-EasyEDA-Edits:SW-SMD_SKSLLAE010-3D" H 5500 5950 50  0001 C CNN
+F 3 "~" H 5500 5950 50  0001 C CNN
+F 4 "C115362" H 5500 5750 50  0001 C CNN "LCSC"
+F 5 "SKSCLDE010" H 5500 5750 50  0001 C CNN "MPN"
+F 6 "ALPS Alpine" H 5500 5750 50  0001 C CNN "Manufacturer"
 	1    5500 5750
-	-1   0    0    1
-$EndComp
-$Comp
-L Switch:SW_Push SW1
-U 1 1 6077308A
-P 5750 5750
-F 0 "SW1" V 5802 5702 50  0000 R CNN
-F 1 "Reset" V 5704 5702 50  0000 R CNN
-F 2 "41-EasyEDA-Edits:SW-SMD_SKSLLAE010-3D" H 5750 5950 50  0001 C CNN
-F 3 "~" H 5750 5950 50  0001 C CNN
-F 4 "C115362" H 5750 5750 50  0001 C CNN "LCSC"
-F 5 "SKSCLDE010" H 5750 5750 50  0001 C CNN "MPN"
-F 6 "ALPS Alpine" H 5750 5750 50  0001 C CNN "Manufacturer"
-	1    5750 5750
-	0    -1   -1   0
-$EndComp
-Wire Wire Line
-	5750 5500 5500 5500
-Wire Wire Line
-	5500 5500 5500 5650
-Wire Wire Line
-	5750 5500 5750 5550
-Wire Wire Line
-	5750 5950 5750 6000
-Wire Wire Line
-	5750 6000 5500 6000
-Wire Wire Line
-	5500 6000 5500 5850
+	0    1    -1   0
+$EndComp
+Wire Wire Line
+	5500 5500 5000 5500
+Wire Wire Line
+	5000 5500 5000 5650
+Wire Wire Line
+	5500 5500 5500 5550
+Wire Wire Line
+	5500 5950 5500 6000
+Wire Wire Line
+	5500 6000 5300 6000
+Wire Wire Line
+	5000 6000 5000 5850
 $Comp
 L power:GND #PWR0101
@@
 	1    0    0    -1
 $EndComp
-Wire Wire Line
-	6250 5950 6250 6100
 $Comp
 L power:GND #PWR0103
 U 1 1 607F1F27
-P 5750 6100
-F 0 "#PWR0103" H 5750 5850 50  0001 C CNN
-F 1 "GND" H 5750 5950 50  0000 C CNN
-F 2 "" H 5750 6100 50  0001 C CNN
-F 3 "" H 5750 6100 50  0001 C CNN
-	1    5750 6100
-	1    0    0    -1
-$EndComp
-Wire Wire Line
-	5750 6000 5750 6100
-Connection ~ 5750 6000
-Wire Wire Line
-	5750 5500 5750 5250
-Connection ~ 5750 5500
+P 5500 6100
+F 0 "#PWR0103" H 5500 5850 50  0001 C CNN
+F 1 "GND" H 5500 5950 50  0000 C CNN
+F 2 "" H 5500 6100 50  0001 C CNN
+F 3 "" H 5500 6100 50  0001 C CNN
+	1    5500 6100
+	1    0    0    -1
+$EndComp
+Wire Wire Line
+	5500 6000 5500 6100
+Connection ~ 5500 6000
+Wire Wire Line
+	5500 5500 5500 5250
+Connection ~ 5500 5500
 Wire Wire Line
 	6250 5550 6250 5250
 Text Label 6250 5250 3    50   ~ 0
 ~BOOT
-Text Label 5750 5250 3    50   ~ 0
+Text Label 5500 5250 3    50   ~ 0
 ~RST
 Text Label 8450 4150 0    50   ~ 0
@@
 	0    1    1    0
 $EndComp
-Connection ~ 1750 3900
+Connection ~ 1750 4000
 Wire Wire Line
 	3100 1600 3150 1600
@@
 Connection ~ 2500 2950
 Wire Wire Line
-	1750 3650 1750 3900
+	1750 3900 1750 4000
 $Comp
 L power:+5V #PWR014
@@
 Wire Wire Line
 	6000 2750 6000 2850
-Wire Wire Line
-	2500 4550 2250 4550
-Connection ~ 2500 4550
-Wire Wire Line
-	2500 4550 2500 4450
 $Comp
 L Device:R_Small R4
@@
 RGB
 Wire Wire Line
-	1750 3900 1750 4100
-Wire Wire Line
-	2000 4100 1950 4100
-Wire Wire Line
-	1950 4100 1950 3900
-Connection ~ 1950 3900
-Wire Wire Line
-	1950 3900 2000 3900
-Wire Wire Line
-	1750 4450 2500 4450
-Wire Wire Line
-	3250 3650 3250 3900
+	1750 4000 1750 4100
+Wire Wire Line
+	2150 4150 2050 4150
+Wire Wire Line
+	2050 4150 2050 4000
+Connection ~ 2050 4000
+Wire Wire Line
+	2050 4000 2150 4000
+Wire Wire Line
+	1750 4500 2100 4500
+Wire Wire Line
+	3250 3900 3250 4000
 NoConn ~ 9750 5650
 Text Label 9700 5650 2    50   ~ 0
@@
 	1    0    0    -1
 $EndComp
+Wire Wire Line
+	6250 5950 6250 6000
+Wire Wire Line
+	5350 5750 5300 5750
+Wire Wire Line
+	5300 5750 5300 6000
+Connection ~ 5300 6000
+Wire Wire Line
+	5300 6000 5000 6000
+Wire Wire Line
+	6100 5750 6050 5750
+Wire Wire Line
+	6050 5750 6050 6000
+Wire Wire Line
+	6050 6000 6250 6000
+Connection ~ 6250 6000
+Wire Wire Line
+	6250 6000 6250 6100
+Connection ~ 2100 4500
+Wire Wire Line
+	2100 4500 2500 4500
+Wire Wire Line
+	2100 4450 2100 4500
+Wire Wire Line
+	2500 4500 2500 4550
 $EndSCHEMATC

Commit message: tweak
Parts:
- added LOGO1: neggles logo, 10-My-Footprints:neggle-logo-0.12, symbol Graphic:SYM_Radio_Waves_Small
- U4: LCSC XC6210B332MR-G -> C47719
Changed lines of the file:
@@
 F 3 "https://www.torexsemi.com/file/xc6220/XC6220.pdf" H 3250 3100 50  0001 C CNN
 F 4 "0;0;-180" H 2500 4100 50  0001 C CNN "JLCPCB_CORRECTION"
-F 5 "XC6210B332MR-G" H 2500 4100 50  0001 C CNN "LCSC"
+F 5 "C47719" H 2500 4100 50  0001 C CNN "LCSC"
 	1    2500 4100
 	1    0    0    -1
@@
 Wire Wire Line
 	2500 4500 2500 4550
+$Comp
+L Graphic:SYM_Radio_Waves_Small LOGO1
+U 1 1 614831D9
+P 6750 1200
+F 0 "LOGO1" H 6750 1340 50  0001 C CNN
+F 1 "neggles logo" H 6750 1075 50  0001 C CNN
+F 2 "10-My-Footprints:neggle-logo-0.12" H 6750 1025 50  0001 C CNN
+F 3 "~" H 6780 1000 50  0001 C CNN
+	1    6750 1200
+	1    0    0    -1
+$EndComp
 $EndSCHEMATC
