File: boards/esp-pmsa-panel.kicad_pcb (KiCad board)
At the start: 2 copper layers, 60 x 120 mm, 183 parts, among them M1 PMSA003, U1 WeMos_D1_mini_Labels, U2 BME68x, U3 OPT3001DNPT

Commit message: Deploying to gh-pages from @ neg2led/esp-pmsa@a730e507301c682fc7d8a88894b304163d40722a 🚀
Parts:
- removed the C4 at (70.8, 144.5)
- removed the C4 at (70.8, 94.0)
- removed the REF** at (50.0, 156.5) (x2)
- removed the REF** at (90.0, 41.5) (x2)
- removed the REF** at (50.0, 41.5) (x2)
- added C8: 10uF, Capacitor_SMD:C_0603_1608Metric_Pad1.05x0.95mm_HandSolder, F.Cu at (53.3, 133.8)
- added C8: 10uF, Capacitor_SMD:C_0603_1608Metric_Pad1.05x0.95mm_HandSolder, F.Cu at (53.3, 83.3)
- added REF**: Fiducial, Fiducial, B.Cu at (50.0, 156.5)
- added REF**: Fiducial, Fiducial, F.Cu at (50.0, 156.5)
- added REF**: Fiducial, Fiducial, B.Cu at (90.0, 41.5)
- added REF**: Fiducial, Fiducial, F.Cu at (90.0, 41.5)
- added REF**: Fiducial, Fiducial, B.Cu at (50.0, 41.5)
- added REF**: Fiducial, Fiducial, F.Cu at (50.0, 41.5)
- C4 (x2): renamed from C8; value 10uF -> 100nF; footprint Capacitor_SMD:C_0603_1608Metric_Pad1.05x0.95mm_HandSolder -> Capacitor_SMD:C_0402_1005Metric
- moved C4 20.5 mm to (70.8, 94.0), turned to 270 degrees
- moved C4 20.5 mm to (70.8, 144.5), turned to 270 degrees
Connections:
- C4 pad 1: Board_2-Board_1-+5V -> Board_2-Board_1-GND
- C4 pad 2: Board_2-Board_1-GND -> Board_2-Board_1-/VCC_SENS
- C4 pad 1: Board_1-Board_1-+5V -> Board_1-Board_1-GND
- C4 pad 2: Board_1-Board_1-GND -> Board_1-Board_1-/VCC_SENS

Commit message: Deploying to gh-pages from @ neg2led/esp-pmsa@060c7214fca1917f5e98065bfc5be80db49c411f 🚀
Parts:
- removed the H3 at (87.5, 103.0)
- removed the H3 at (87.5, 52.5)
- removed the REF** at (50.0, 156.5) (x2)
- removed the REF** at (90.0, 41.5) (x2)
- removed the REF** at (50.0, 41.5) (x2)
- added REF**: Fiducial, Fiducial, B.Cu at (50.0, 156.5)
- added REF**: Fiducial, Fiducial, F.Cu at (50.0, 156.5)
- added REF**: Fiducial, Fiducial, B.Cu at (90.0, 41.5)
- added REF**: Fiducial, Fiducial, F.Cu at (90.0, 41.5)
- added REF**: Fiducial, Fiducial, B.Cu at (50.0, 41.5)
- added REF**: Fiducial, Fiducial, F.Cu at (50.0, 41.5)
- added U3: OPT3001DNPT, 11-My-Edits:MultiALS-LTR303-TIOPT3K, F.Cu at (86.3, 119.0)
- added U3: OPT3001DNPT, 11-My-Edits:MultiALS-LTR303-TIOPT3K, F.Cu at (86.3, 68.5)
- H3 (x2): renamed from U3; value OPT3001DNPT -> MP; footprint 11-My-Edits:MultiALS-LTR303-TIOPT3K -> MountingHole:MountingHole_2.2mm_M2_DIN965_Pad_TopBottom
- moved H3 16.0 mm to (87.5, 103.0), turned to 0 degrees
- moved H3 16.0 mm to (87.5, 52.5), turned to 0 degrees
Connections:
- H3 pad 1: Board_2-Board_1-/VCC_SENS -> Board_2-Board_1-GND
- H3 pad 1: Board_1-Board_1-/VCC_SENS -> Board_1-Board_1-GND

Commit message: Deploying to gh-pages from @ neg2led/esp-pmsa@5249862c854155dbbe1c443dd720162530209050 🚀
Parts:
- removed the H1 at (52.5, 52.5)
- removed the H3 at (87.5, 103.0)
- removed the REF** at (50.0, 156.5) (x2)
- removed the REF** at (90.0, 41.5) (x2)
- removed the REF** at (50.0, 41.5) (x2)
- removed the U1 at (70.0, 121.5)
- removed the U2 at (70.0, 94.5)
- added REF**: NPTH, NPTH, F.Cu at (79.6, 90.5)
- added REF**: NPTH, NPTH, F.Cu at (67.5, 53.7)
- added REF**: Fiducial, Fiducial, B.Cu at (50.0, 156.5)
- added REF**: Fiducial, Fiducial, F.Cu at (50.0, 156.5)
- added REF**: Fiducial, Fiducial, B.Cu at (90.0, 41.5)
- added REF**: Fiducial, Fiducial, F.Cu at (90.0, 41.5)
- added REF**: Fiducial, Fiducial, B.Cu at (50.0, 41.5)
- added REF**: Fiducial, Fiducial, F.Cu at (50.0, 41.5)
- added REF**: NPTH, NPTH, F.Cu at (50.2, 64.4)
- added REF**: NPTH, NPTH, F.Cu at (60.4, 141.0)
- H1, H3: renamed from REF**; value NPTH -> MP; footprint NPTH -> MountingHole:MountingHole_2.2mm_M2_DIN965_Pad_TopBottom
- U1: renamed from REF**; value NPTH -> WeMos_D1_mini_Labels; footprint NPTH -> 11-My-Edits:WEMOS_D1_mini
- U2: renamed from REF**; value NPTH -> BME68x; footprint NPTH -> 11-My-Edits:Bosch_LGA-8_3x3mm_P0.8mm_ClockwisePinNumbering; moved to B.Cu
- moved U1 60.4 mm to (70.0, 121.5)
- moved H3 46.7 mm to (87.5, 103.0)
- moved H1 15.1 mm to (52.5, 52.5)
- moved U2 10.4 mm to (70.0, 94.5), turned to 90 degrees
