File: boards/esp-pmsa-panel.kicad_pcb (KiCad board)
At the start: 2 copper layers, 60 x 120 mm, 183 parts, among them M1 PMSA003, U1 WeMos_D1_mini_Labels, U2 BME68x, U3 OPT3001DNPT

Commit message: Deploying to gh-pages from @ neg2led/esp-pmsa@e03a36f01e21f29b520752c6169685313d9a0f2f 🚀
Parts:
- removed the C3 at (69.3, 144.5)
- removed the C3 at (69.3, 94.0)
- removed the C4 at (70.8, 144.5)
- removed the C4 at (70.8, 94.0)
- removed the C7 at (53.3, 135.3)
- removed the C7 at (53.3, 84.8)
- removed the C8 at (53.3, 133.8)
- removed the C8 at (53.3, 83.3)
- removed the H2 at (87.5, 145.5)
- removed the H2 at (87.5, 95.0)
- removed the H3 at (87.5, 103.0)
- removed the H3 at (87.5, 52.5)
- removed the H4 at (52.5, 145.5)
- removed the H4 at (52.5, 95.0)
- removed the M1 at (70.0, 123.0)
- removed the M1 at (70.0, 72.5)
- removed the REF** at (89.8, 138.6)
- removed the REF** at (89.8, 123.8)
- removed the REF** at (72.5, 104.3)
- removed the REF** at (71.5, 104.3)
- removed the REF** at (70.5, 104.3)
- removed the REF** at (69.5, 104.3)
- removed the REF** at (68.5, 104.3)
- removed the REF** at (67.5, 104.3)
- removed the REF** at (62.5, 104.3)
- removed the REF** at (61.5, 104.3)
- removed the REF** at (60.5, 104.3)
- removed the REF** at (59.5, 104.3)
- removed the REF** at (89.8, 122.8)
- removed the REF** at (58.5, 104.3)
- removed the REF** at (57.5, 104.3)
- removed the REF** at (77.5, 90.5)
- removed the REF** at (78.6, 90.5)
- removed the REF** at (79.6, 90.5)
- removed the REF** at (80.7, 90.5)
- removed the REF** at (81.8, 90.7)
- removed the REF** at (82.7, 91.3)
- removed the REF** at (67.7, 94.1)
- removed the REF** at (67.8, 95.2)
- removed the REF** at (89.8, 121.8)
- removed the REF** at (68.1, 96.2)
- removed the REF** at (68.9, 96.7)
- removed the REF** at (70.0, 96.8)
- removed the REF** at (71.1, 96.7)
- removed the REF** at (71.9, 96.2)
- removed the REF** at (72.2, 95.2)
- removed the REF** at (72.3, 94.1)
- removed the REF** at (57.3, 91.3)
- removed the REF** at (58.2, 90.7)
- removed the REF** at (59.3, 90.5)
- removed the REF** at (89.8, 114.9)
- removed the REF** at (60.4, 90.5)
- removed the REF** at (61.4, 90.5)
- removed the REF** at (62.5, 90.5)
- removed the REF** at (82.5, 53.7)
- removed the REF** at (81.5, 53.7)
- removed the REF** at (80.5, 53.7)
- removed the REF** at (79.5, 53.7)
- removed the REF** at (78.5, 53.7)
- removed the REF** at (77.5, 53.7)
- removed the REF** at (72.5, 53.7)
- removed the REF** at (89.8, 113.9)
- removed the REF** at (71.5, 53.7)
- removed the REF** at (70.5, 53.7)
- removed the REF** at (69.5, 53.7)
- removed the REF** at (68.5, 53.7)
- removed the REF** at (67.5, 53.7)
- removed the REF** at (62.5, 53.7)
- removed the REF** at (61.5, 53.7)
- removed the REF** at (60.5, 53.7)
- removed the REF** at (59.5, 53.7)
- removed the REF** at (58.5, 53.7)
- removed the REF** at (89.8, 112.9)
- removed the REF** at (57.5, 53.7)
- removed the REF** at (45.0, 156.5)
- removed the REF** at (95.0, 41.5)
- removed the REF** at (45.0, 41.5)
- removed the REF** at (50.0, 156.5) (x2)
- removed the REF** at (90.0, 41.5) (x2)
- removed the REF** at (50.0, 41.5) (x2)
- removed the REF** at (89.8, 111.9)
- removed the REF** at (89.8, 110.9)
- removed the REF** at (89.8, 109.9)
- removed the REF** at (50.2, 133.6)
- removed the REF** at (89.8, 137.6)
- removed the REF** at (50.2, 134.6)
- removed the REF** at (50.2, 135.6)
- removed the REF** at (50.2, 136.6)
- removed the REF** at (50.2, 137.6)
- removed the REF** at (50.2, 138.6)
- removed the REF** at (50.2, 121.8)
- removed the REF** at (50.2, 122.8)
- removed the REF** at (50.2, 123.8)
- removed the REF** at (50.2, 124.8)
- removed the REF** at (50.2, 125.8)
- removed the REF** at (89.8, 136.6)
- removed the REF** at (50.2, 126.8)
- removed the REF** at (50.2, 109.9)
- removed the REF** at (50.2, 110.9)
- removed the REF** at (50.2, 111.9)
- removed the REF** at (50.2, 112.9)
- removed the REF** at (50.2, 113.9)
- removed the REF** at (50.2, 114.9)
- removed the REF** at (89.8, 88.1)
- removed the REF** at (89.8, 87.1)
- removed the REF** at (89.8, 86.1)
- removed the REF** at (89.8, 135.6)
- removed the REF** at (89.8, 85.1)
- removed the REF** at (89.8, 84.1)
- removed the REF** at (89.8, 83.1)
- removed the REF** at (89.8, 76.3)
- removed the REF** at (89.8, 75.3)
- removed the REF** at (89.8, 74.3)
- removed the REF** at (89.8, 73.3)
- removed the REF** at (89.8, 72.3)
- removed the REF** at (89.8, 71.3)
- removed the REF** at (89.8, 64.4)
- removed the REF** at (89.8, 134.6)
- removed the REF** at (89.8, 63.4)
- removed the REF** at (89.8, 62.4)
- removed the REF** at (89.8, 61.4)
- removed the REF** at (89.8, 60.4)
- removed the REF** at (89.8, 59.4)
- removed the REF** at (50.2, 83.1)
- removed the REF** at (50.2, 84.1)
- removed the REF** at (50.2, 85.1)
- removed the REF** at (50.2, 86.1)
- removed the REF** at (50.2, 87.1)
- removed the REF** at (89.8, 133.6)
- removed the REF** at (50.2, 88.1)
- removed the REF** at (50.2, 71.3)
- removed the REF** at (50.2, 72.3)
- removed the REF** at (50.2, 73.3)
- removed the REF** at (50.2, 74.3)
- removed the REF** at (50.2, 75.3)
- removed the REF** at (50.2, 76.3)
- removed the REF** at (50.2, 59.4)
- removed the REF** at (50.2, 60.4)
- removed the REF** at (50.2, 61.4)
- removed the REF** at (89.8, 126.8)
- removed the REF** at (50.2, 62.4)
- removed the REF** at (50.2, 63.4)
- removed the REF** at (50.2, 64.4)
- removed the REF** at (77.5, 141.0)
- removed the REF** at (78.6, 141.0)
- removed the REF** at (79.6, 141.0)
- removed the REF** at (80.7, 141.0)
- removed the REF** at (81.8, 141.2)
- removed the REF** at (82.7, 141.8)
- removed the REF** at (67.7, 144.6)
- removed the REF** at (89.8, 125.8)
- removed the REF** at (67.8, 145.7)
- removed the REF** at (68.1, 146.7)
- removed the REF** at (68.9, 147.2)
- removed the REF** at (70.0, 147.3)
- removed the REF** at (71.1, 147.2)
- removed the REF** at (71.9, 146.7)
- removed the REF** at (72.2, 145.7)
- removed the REF** at (72.3, 144.6)
- removed the REF** at (57.3, 141.8)
- removed the REF** at (58.2, 141.2)
- removed the REF** at (89.8, 124.8)
- removed the REF** at (59.3, 141.0)
- removed the REF** at (60.4, 141.0)
- removed the REF** at (61.4, 141.0)
- removed the REF** at (62.5, 141.0)
- removed the REF** at (82.5, 104.3)
- removed the REF** at (81.5, 104.3)
- removed the REF** at (80.5, 104.3)
- removed the REF** at (79.5, 104.3)
- removed the REF** at (78.5, 104.3)
- removed the REF** at (77.5, 104.3)
- removed the U1 at (70.0, 121.5)
- removed the U1 at (70.0, 71.0)
- removed the U2 at (70.0, 145.0)
- removed the U2 at (70.0, 94.5)
- removed the U3 at (86.3, 119.0)
- removed the U3 at (86.3, 68.5)
- added C1: 10u, Capacitor_SMD:C_0402_1005Metric, F.Cu at (68.1, 131.9)
- added C1: 10u, Capacitor_SMD:C_0402_1005Metric, F.Cu at (68.1, 78.9)
- added C2: 10u, Capacitor_SMD:C_0402_1005Metric, F.Cu at (63.4, 131.1)
- added C2: 10u, Capacitor_SMD:C_0402_1005Metric, F.Cu at (63.4, 78.1)
- added C3: 1u, Capacitor_SMD:C_0402_1005Metric, F.Cu at (75.0, 129.5)
- added C3: 1u, Capacitor_SMD:C_0402_1005Metric, F.Cu at (75.0, 76.5)
- added C4: 0.1u, Capacitor_SMD:C_0402_1005Metric, F.Cu at (70.5, 143.3)
- added C4: 0.1u, Capacitor_SMD:C_0402_1005Metric, F.Cu at (70.5, 90.3)
- added C5: 1u, Capacitor_SMD:C_0402_1005Metric, F.Cu at (72.0, 129.5)
- added C5: 1u, Capacitor_SMD:C_0402_1005Metric, F.Cu at (72.0, 76.5)
- added C6: 0.1u, Capacitor_SMD:C_0402_1005Metric, F.Cu at (64.0, 143.3)
- added C6: 0.1u, Capacitor_SMD:C_0402_1005Metric, F.Cu at (64.0, 90.3)
- added C7: 10u, Capacitor_SMD:C_0603_1608Metric_Pad1.05x0.95mm_HandSolder, F.Cu at (58.3, 139.9)
- added C7: 10u, Capacitor_SMD:C_0603_1608Metric_Pad1.05x0.95mm_HandSolder, F.Cu at (58.3, 86.9)
- added C8: 10u, Capacitor_SMD:C_0603_1608Metric_Pad1.05x0.95mm_HandSolder, F.Cu at (58.3, 141.4)
- added C8: 10u, Capacitor_SMD:C_0603_1608Metric_Pad1.05x0.95mm_HandSolder, F.Cu at (58.3, 88.4)
- added C9: 0.1u, Capacitor_SMD:C_0402_1005Metric, F.Cu at (59.5, 115.0)
- added C9: 0.1u, Capacitor_SMD:C_0402_1005Metric, F.Cu at (59.5, 62.0)
- added D1: APA104-12-3535, 21-SnapEDA-zip:LED_APA104-12-3535, F.Cu at (87.5, 125.5)
- added D1: APA104-12-3535, 21-SnapEDA-zip:LED_APA104-12-3535, F.Cu at (87.5, 72.5)
- added H2: MP, MountingHole:MountingHole_2.2mm_M2_DIN965_Pad_TopBottom, F.Cu at (90.5, 150.5)
- added H2: MP, MountingHole:MountingHole_2.2mm_M2_DIN965_Pad_TopBottom, F.Cu at (90.5, 97.5)
- added H3: MP, MountingHole:MountingHole_2.2mm_M2_DIN965_Pad_TopBottom, F.Cu at (90.5, 105.5)
- added H3: MP, MountingHole:MountingHole_2.2mm_M2_DIN965_Pad_TopBottom, F.Cu at (90.5, 52.5)
- added H4: MP, MountingHole:MountingHole_2.2mm_M2_DIN965_Pad_TopBottom, F.Cu at (52.5, 150.5)
- added H4: MP, MountingHole:MountingHole_2.2mm_M2_DIN965_Pad_TopBottom, F.Cu at (52.5, 97.5)
- added J1: USB_C_Receptacle_USB2.0_304S-ACP16, 41-EasyEDA-Edits:USB-C-SMD_TYPEC-304S-ACP16, F.Cu at (80.0, 141.1)
- added J1: USB_C_Receptacle_USB2.0_304S-ACP16, 41-EasyEDA-Edits:USB-C-SMD_TYPEC-304S-ACP16, F.Cu at (80.0, 88.1)
- added J2: ESP-PROG, 11-My-Edits:TC2030_IDCBox_2x03_P1.25mm_Vertical_3D, F.Cu at (87.5, 113.1)
- added J2: ESP-PROG, 11-My-Edits:TC2030_IDCBox_2x03_P1.25mm_Vertical_3D, F.Cu at (87.5, 60.1)
- added M1: PMSA003, 12-Collected-Footprints:PMSA003, B.Cu at (71.5, 125.5)
- added M1: PMSA003, 12-Collected-Footprints:PMSA003, B.Cu at (71.5, 72.5)
- added R1: 4k7, Resistor_SMD:R_0402_1005Metric, F.Cu at (59.0, 123.2)
- added R1: 4k7, Resistor_SMD:R_0402_1005Metric, F.Cu at (59.0, 70.2)
- added R2: 4k7, Resistor_SMD:R_0402_1005Metric, F.Cu at (59.0, 121.8)
- added R2: 4k7, Resistor_SMD:R_0402_1005Metric, F.Cu at (59.0, 68.8)
- added R3: 5k1, Resistor_SMD:R_0402_1005Metric, F.Cu at (89.0, 145.8)
- added R3: 5k1, Resistor_SMD:R_0402_1005Metric, F.Cu at (89.0, 92.8)
- added R4: 5k1, Resistor_SMD:R_0402_1005Metric, F.Cu at (89.0, 144.7)
- added R4: 5k1, Resistor_SMD:R_0402_1005Metric, F.Cu at (89.0, 91.7)
- added REF**: NPTH, NPTH, F.Cu at (92.8, 143.0)
- added REF**: NPTH, NPTH, F.Cu at (92.8, 127.5)
- added REF**: NPTH, NPTH, F.Cu at (79.8, 106.8)
- added REF**: NPTH, NPTH, F.Cu at (74.0, 106.8)
- added REF**: NPTH, NPTH, F.Cu at (73.0, 106.8)
- added REF**: NPTH, NPTH, F.Cu at (72.0, 106.8)
- added REF**: NPTH, NPTH, F.Cu at (71.0, 106.8)
- added REF**: NPTH, NPTH, F.Cu at (70.0, 106.8)
- added REF**: NPTH, NPTH, F.Cu at (69.0, 106.8)
- added REF**: NPTH, NPTH, F.Cu at (63.3, 106.8)
- added REF**: NPTH, NPTH, F.Cu at (62.3, 106.8)
- added REF**: NPTH, NPTH, F.Cu at (61.3, 106.8)
- added REF**: NPTH, NPTH, F.Cu at (92.8, 126.5)
- added REF**: NPTH, NPTH, F.Cu at (60.3, 106.8)
- added REF**: NPTH, NPTH, F.Cu at (59.3, 106.8)
- added REF**: NPTH, NPTH, F.Cu at (58.3, 106.8)
- added REF**: NPTH, NPTH, F.Cu at (79.8, 93.0)
- added REF**: NPTH, NPTH, F.Cu at (80.8, 93.0)
- added REF**: NPTH, NPTH, F.Cu at (81.8, 93.0)
- added REF**: NPTH, NPTH, F.Cu at (82.8, 93.0)
- added REF**: NPTH, NPTH, F.Cu at (83.8, 93.0)
- added REF**: NPTH, NPTH, F.Cu at (84.8, 93.0)
- added REF**: NPTH, NPTH, F.Cu at (68.9, 99.1)
- added REF**: NPTH, NPTH, F.Cu at (92.8, 125.5)
- added REF**: NPTH, NPTH, F.Cu at (69.5, 98.3)
- added REF**: NPTH, NPTH, F.Cu at (69.6, 97.3)
- added REF**: NPTH, NPTH, F.Cu at (70.1, 96.3)
- added REF**: NPTH, NPTH, F.Cu at (70.8, 95.6)
- added REF**: NPTH, NPTH, F.Cu at (71.5, 94.9)
- added REF**: NPTH, NPTH, F.Cu at (72.2, 94.1)
- added REF**: NPTH, NPTH, F.Cu at (73.0, 93.4)
- added REF**: NPTH, NPTH, F.Cu at (74.0, 93.1)
- added REF**: NPTH, NPTH, F.Cu at (58.3, 93.0)
- added REF**: NPTH, NPTH, F.Cu at (59.3, 93.0)
- added REF**: NPTH, NPTH, F.Cu at (92.8, 118.0)
- added REF**: NPTH, NPTH, F.Cu at (60.3, 93.0)
- added REF**: NPTH, NPTH, F.Cu at (61.2, 93.3)
- added REF**: NPTH, NPTH, F.Cu at (62.0, 93.9)
- added REF**: NPTH, NPTH, F.Cu at (62.7, 94.6)
- added REF**: NPTH, NPTH, F.Cu at (63.4, 95.3)
- added REF**: NPTH, NPTH, F.Cu at (84.8, 53.7)
- added REF**: NPTH, NPTH, F.Cu at (83.8, 53.7)
- added REF**: NPTH, NPTH, F.Cu at (82.8, 53.7)
- added REF**: NPTH, NPTH, F.Cu at (81.8, 53.7)
- added REF**: NPTH, NPTH, F.Cu at (80.8, 53.7)
- added REF**: NPTH, NPTH, F.Cu at (92.8, 117.0)
- added REF**: NPTH, NPTH, F.Cu at (79.8, 53.7)
- added REF**: NPTH, NPTH, F.Cu at (74.0, 53.7)
- added REF**: NPTH, NPTH, F.Cu at (73.0, 53.7)
- added REF**: NPTH, NPTH, F.Cu at (72.0, 53.7)
- added REF**: NPTH, NPTH, F.Cu at (71.0, 53.7)
- added REF**: NPTH, NPTH, F.Cu at (70.0, 53.7)
- added REF**: NPTH, NPTH, F.Cu at (69.0, 53.7)
- added REF**: NPTH, NPTH, F.Cu at (63.3, 53.7)
- added REF**: NPTH, NPTH, F.Cu at (62.3, 53.7)
- added REF**: NPTH, NPTH, F.Cu at (61.3, 53.7)
- added REF**: NPTH, NPTH, F.Cu at (92.8, 116.0)
- added REF**: NPTH, NPTH, F.Cu at (60.3, 53.7)
- added REF**: NPTH, NPTH, F.Cu at (59.3, 53.7)
- added REF**: NPTH, NPTH, F.Cu at (58.3, 53.7)
- added REF**: NPTH, NPTH, F.Cu at (46.5, 159.0)
- added REF**: NPTH, NPTH, F.Cu at (96.5, 44.0)
- added REF**: NPTH, NPTH, F.Cu at (46.5, 44.0)
- added REF**: Fiducial, Fiducial, B.Cu at (51.5, 159.0)
- added REF**: Fiducial, Fiducial, F.Cu at (51.5, 159.0)
- added REF**: Fiducial, Fiducial, B.Cu at (91.5, 44.0)
- added REF**: Fiducial, Fiducial, F.Cu at (91.5, 44.0)
- added REF**: NPTH, NPTH, F.Cu at (92.8, 115.0)
- added REF**: Fiducial, Fiducial, B.Cu at (51.5, 44.0)
- added REF**: Fiducial, Fiducial, F.Cu at (51.5, 44.0)
- added REF**: NPTH, NPTH, F.Cu at (92.8, 114.0)
- added REF**: NPTH, NPTH, F.Cu at (92.8, 113.0)
- added REF**: NPTH, NPTH, F.Cu at (50.2, 138.0)
- added REF**: NPTH, NPTH, F.Cu at (92.8, 142.0)
- added REF**: NPTH, NPTH, F.Cu at (50.2, 139.0)
- added REF**: NPTH, NPTH, F.Cu at (50.2, 140.0)
- added REF**: NPTH, NPTH, F.Cu at (50.2, 141.0)
- added REF**: NPTH, NPTH, F.Cu at (50.2, 142.0)
- added REF**: NPTH, NPTH, F.Cu at (50.2, 143.0)
- added REF**: NPTH, NPTH, F.Cu at (50.2, 125.5)
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Routing:
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- removed copper zone on B.Cu, net Board_1-Board_1-GND
- removed copper zone on F.Cu, net Board_1-Board_1-GND
- removed copper zone on B.Cu, net Board_2-Board_1-GND
- removed copper zone on F.Cu, net Board_2-Board_1-GND
Other:
- outline, holes or cut-outs redrawn
- board text added: "Boot"
- board text added: "Reset"
- board text removed: "vriska did nothing wrong"

Commit message: Deploying to gh-pages from @ neg2led/esp-pmsa@1a288ce33808fbc405a6c24b3a385c7c225d67b1 🚀
Parts:
- removed the C1 at (68.1, 131.9)
- removed the C1 at (68.1, 78.9)
- removed the C2 at (63.4, 131.1)
- removed the C2 at (63.4, 78.1)
- removed the C4 at (70.5, 143.3)
- removed the C4 at (70.5, 90.3)
- removed the C6 at (64.0, 143.3)
- removed the C6 at (64.0, 90.3)
- removed the C9 at (59.5, 115.0)
- removed the C9 at (59.5, 62.0)
- removed the R1 at (59.0, 123.2)
- removed the R1 at (59.0, 70.2)
- removed the R2 at (59.0, 121.8)
- removed the R2 at (59.0, 68.8)
- removed the REF** at (92.8, 143.0)
- removed the REF** at (92.8, 127.5)
- removed the REF** at (79.8, 106.8)
- removed the REF** at (74.0, 106.8)
- removed the REF** at (73.0, 106.8)
- removed the REF** at (72.0, 106.8)
- removed the REF** at (71.0, 106.8)
- removed the REF** at (70.0, 106.8)
- removed the REF** at (69.0, 106.8)
- removed the REF** at (63.3, 106.8)
- removed the REF** at (62.3, 106.8)
- removed the REF** at (61.3, 106.8)
- removed the REF** at (92.8, 126.5)
- removed the REF** at (60.3, 106.8)
- removed the REF** at (59.3, 106.8)
- removed the REF** at (58.3, 106.8)
- removed the REF** at (79.8, 93.0)
- removed the REF** at (80.8, 93.0)
- removed the REF** at (81.8, 93.0)
- removed the REF** at (82.8, 93.0)
- removed the REF** at (83.8, 93.0)
- removed the REF** at (84.8, 93.0)
- removed the REF** at (68.9, 99.1)
- removed the REF** at (92.8, 125.5)
- removed the REF** at (69.5, 98.3)
- removed the REF** at (69.6, 97.3)
- removed the REF** at (70.1, 96.3)
- removed the REF** at (70.8, 95.6)
- removed the REF** at (71.5, 94.9)
- removed the REF** at (72.2, 94.1)
- removed the REF** at (73.0, 93.4)
- removed the REF** at (74.0, 93.1)
- removed the REF** at (58.3, 93.0)
- removed the REF** at (59.3, 93.0)
- removed the REF** at (92.8, 118.0)
- removed the REF** at (60.3, 93.0)
- removed the REF** at (61.2, 93.3)
- removed the REF** at (62.0, 93.9)
- removed the REF** at (62.7, 94.6)
- removed the REF** at (63.4, 95.3)
- removed the REF** at (84.8, 53.7)
- removed the REF** at (83.8, 53.7)
- removed the REF** at (82.8, 53.7)
- removed the REF** at (81.8, 53.7)
- removed the REF** at (80.8, 53.7)
- removed the REF** at (92.8, 117.0)
- removed the REF** at (79.8, 53.7)
- removed the REF** at (74.0, 53.7)
- removed the REF** at (73.0, 53.7)
- removed the REF** at (72.0, 53.7)
- removed the REF** at (71.0, 53.7)
- removed the REF** at (70.0, 53.7)
- removed the REF** at (69.0, 53.7)
- removed the REF** at (63.3, 53.7)
- removed the REF** at (62.3, 53.7)
- removed the REF** at (61.3, 53.7)
- removed the REF** at (92.8, 116.0)
- removed the REF** at (60.3, 53.7)
- removed the REF** at (59.3, 53.7)
- removed the REF** at (58.3, 53.7)
- removed the REF** at (46.5, 159.0)
- removed the REF** at (96.5, 44.0)
- removed the REF** at (46.5, 44.0)
- removed the REF** at (51.5, 159.0) (x2)
- removed the REF** at (91.5, 44.0) (x2)
- removed the REF** at (92.8, 115.0)
- removed the REF** at (51.5, 44.0) (x2)
- removed the REF** at (92.8, 114.0)
- removed the REF** at (92.8, 113.0)
- removed the REF** at (50.2, 138.0)
- removed the REF** at (92.8, 142.0)
- removed the REF** at (50.2, 139.0)
- removed the REF** at (50.2, 140.0)
- removed the REF** at (50.2, 141.0)
- removed the REF** at (50.2, 142.0)
- removed the REF** at (50.2, 143.0)
- removed the REF** at (50.2, 125.5)
- removed the REF** at (50.2, 126.5)
- removed the REF** at (50.2, 127.5)
- removed the REF** at (50.2, 128.5)
- removed the REF** at (50.2, 129.5)
- removed the REF** at (92.8, 141.0)
- removed the REF** at (50.2, 130.5)
- removed the REF** at (50.2, 113.0)
- removed the REF** at (50.2, 114.0)
- removed the REF** at (50.2, 115.0)
- removed the REF** at (50.2, 116.0)
- removed the REF** at (50.2, 117.0)
- removed the REF** at (50.2, 118.0)
- removed the REF** at (92.8, 90.0)
- removed the REF** at (92.8, 89.0)
- removed the REF** at (92.8, 88.0)
- removed the REF** at (92.8, 140.0)
- removed the REF** at (92.8, 87.0)
- removed the REF** at (92.8, 86.0)
- removed the REF** at (92.8, 85.0)
- removed the REF** at (92.8, 77.5)
- removed the REF** at (92.8, 76.5)
- removed the REF** at (92.8, 75.5)
- removed the REF** at (92.8, 74.5)
- removed the REF** at (92.8, 73.5)
- removed the REF** at (92.8, 72.5)
- removed the REF** at (92.8, 65.0)
- removed the REF** at (92.8, 139.0)
- removed the REF** at (92.8, 64.0)
- removed the REF** at (92.8, 63.0)
- removed the REF** at (92.8, 62.0)
- removed the REF** at (92.8, 61.0)
- removed the REF** at (92.8, 60.0)
- removed the REF** at (50.2, 85.0)
- removed the REF** at (50.2, 86.0)
- removed the REF** at (50.2, 87.0)
- removed the REF** at (50.2, 88.0)
- removed the REF** at (50.2, 89.0)
- removed the REF** at (92.8, 138.0)
- removed the REF** at (50.2, 90.0)
- removed the REF** at (50.2, 72.5)
- removed the REF** at (50.2, 73.5)
- removed the REF** at (50.2, 74.5)
- removed the REF** at (50.2, 75.5)
- removed the REF** at (50.2, 76.5)
- removed the REF** at (50.2, 77.5)
- removed the REF** at (50.2, 60.0)
- removed the REF** at (50.2, 61.0)
- removed the REF** at (50.2, 62.0)
- removed the REF** at (92.8, 130.5)
- removed the REF** at (50.2, 63.0)
- removed the REF** at (50.2, 64.0)
- removed the REF** at (50.2, 65.0)
- removed the REF** at (79.8, 146.0)
- removed the REF** at (80.8, 146.0)
- removed the REF** at (81.8, 146.0)
- removed the REF** at (82.8, 146.0)
- removed the REF** at (83.8, 146.0)
- removed the REF** at (84.8, 146.0)
- removed the REF** at (68.9, 152.1)
- removed the REF** at (92.8, 129.5)
- removed the REF** at (69.5, 151.3)
- removed the REF** at (69.6, 150.3)
- removed the REF** at (70.1, 149.3)
- removed the REF** at (70.8, 148.6)
- removed the REF** at (71.5, 147.9)
- removed the REF** at (72.2, 147.1)
- removed the REF** at (73.0, 146.4)
- removed the REF** at (74.0, 146.1)
- removed the REF** at (58.3, 146.0)
- removed the REF** at (59.3, 146.0)
- removed the REF** at (92.8, 128.5)
- removed the REF** at (60.3, 146.0)
- removed the REF** at (61.2, 146.3)
- removed the REF** at (62.0, 146.9)
- removed the REF** at (62.7, 147.6)
- removed the REF** at (63.4, 148.3)
- removed the REF** at (84.8, 106.8)
- removed the REF** at (83.8, 106.8)
- removed the REF** at (82.8, 106.8)
- removed the REF** at (81.8, 106.8)
- removed the REF** at (80.8, 106.8)
- removed the U2 at (67.3, 150.1)
- removed the U2 at (67.3, 97.1)
- removed the U3 at (67.2, 150.1)
- removed the U3 at (67.2, 97.1)
- removed the U4 at (65.8, 131.5)
- removed the U4 at (65.8, 78.5)
- added C1: 10u, Capacitor_SMD:C_0402_1005Metric, F.Cu at (62.3, 132.5)
- added C1: 10u, Capacitor_SMD:C_0402_1005Metric, F.Cu at (62.3, 79.5)
- added C2: 10u, Capacitor_SMD:C_0402_1005Metric, F.Cu at (62.3, 130.5)
- added C2: 10u, Capacitor_SMD:C_0402_1005Metric, F.Cu at (62.3, 77.5)
- added C4: 0.1u, Capacitor_SMD:C_0402_1005Metric, F.Cu at (70.8, 147.5)
- added C4: 0.1u, Capacitor_SMD:C_0402_1005Metric, F.Cu at (70.8, 94.5)
- added C6: 0.1u, Capacitor_SMD:C_0402_1005Metric, F.Cu at (69.5, 141.7)
- added C6: 0.1u, Capacitor_SMD:C_0402_1005Metric, F.Cu at (69.5, 88.7)
- added C9: 0.1u, Capacitor_SMD:C_0402_1005Metric, F.Cu at (60.5, 115.5)
- added C9: 0.1u, Capacitor_SMD:C_0402_1005Metric, F.Cu at (60.5, 62.5)
- added LOGO1: neggles logo, 10-My-Footprints:neggle-logo-0.12, F.Cu at (81.5, 131.5)
- added LOGO1: neggles logo, 10-My-Footprints:neggle-logo-0.12, F.Cu at (81.5, 78.5)
- added R1: 4k7, Resistor_SMD:R_0402_1005Metric, F.Cu at (60.5, 123.5)
- added R1: 4k7, Resistor_SMD:R_0402_1005Metric, F.Cu at (60.5, 70.5)
- added R2: 4k7, Resistor_SMD:R_0402_1005Metric, F.Cu at (60.5, 121.5)
- added R2: 4k7, Resistor_SMD:R_0402_1005Metric, F.Cu at (60.5, 68.5)
- added REF**: NPTH, NPTH, F.Cu at (92.8, 143.0)
- added REF**: NPTH, NPTH, F.Cu at (92.8, 127.5)
- added REF**: NPTH, NPTH, F.Cu at (79.8, 106.8)
- added REF**: NPTH, NPTH, F.Cu at (74.0, 106.8)
- added REF**: NPTH, NPTH, F.Cu at (73.0, 106.8)
- added REF**: NPTH, NPTH, F.Cu at (72.0, 106.8)
- added REF**: NPTH, NPTH, F.Cu at (71.0, 106.8)
- added REF**: NPTH, NPTH, F.Cu at (70.0, 106.8)
- added REF**: NPTH, NPTH, F.Cu at (69.0, 106.8)
- added REF**: NPTH, NPTH, F.Cu at (63.3, 106.8)
- added REF**: NPTH, NPTH, F.Cu at (62.3, 106.8)
- added REF**: NPTH, NPTH, F.Cu at (61.3, 106.8)
- added REF**: NPTH, NPTH, F.Cu at (92.8, 126.5)
- added REF**: NPTH, NPTH, F.Cu at (60.3, 106.8)
- added REF**: NPTH, NPTH, F.Cu at (59.3, 106.8)
- added REF**: NPTH, NPTH, F.Cu at (58.3, 106.8)
- added REF**: NPTH, NPTH, F.Cu at (79.8, 93.0)
- added REF**: NPTH, NPTH, F.Cu at (80.8, 93.0)
- added REF**: NPTH, NPTH, F.Cu at (81.8, 93.0)
- added REF**: NPTH, NPTH, F.Cu at (82.8, 93.0)
- added REF**: NPTH, NPTH, F.Cu at (83.8, 93.0)
- added REF**: NPTH, NPTH, F.Cu at (84.8, 93.0)
- added REF**: NPTH, NPTH, F.Cu at (68.9, 99.1)
- added REF**: NPTH, NPTH, F.Cu at (92.8, 125.5)
- added REF**: NPTH, NPTH, F.Cu at (69.5, 98.3)
- added REF**: NPTH, NPTH, F.Cu at (69.6, 97.3)
- added REF**: NPTH, NPTH, F.Cu at (70.1, 96.3)
- added REF**: NPTH, NPTH, F.Cu at (70.8, 95.6)
- added REF**: NPTH, NPTH, F.Cu at (71.5, 94.9)
- added REF**: NPTH, NPTH, F.Cu at (72.2, 94.1)
- added REF**: NPTH, NPTH, F.Cu at (73.0, 93.4)
- added REF**: NPTH, NPTH, F.Cu at (74.0, 93.1)
- added REF**: NPTH, NPTH, F.Cu at (58.3, 93.0)
- added REF**: NPTH, NPTH, F.Cu at (59.3, 93.0)
- added REF**: NPTH, NPTH, F.Cu at (92.8, 118.0)
- added REF**: NPTH, NPTH, F.Cu at (60.3, 93.0)
- added REF**: NPTH, NPTH, F.Cu at (61.2, 93.3)
- added REF**: NPTH, NPTH, F.Cu at (62.0, 93.9)
- added REF**: NPTH, NPTH, F.Cu at (62.7, 94.6)
- added REF**: NPTH, NPTH, F.Cu at (63.4, 95.3)
- added REF**: NPTH, NPTH, F.Cu at (84.8, 53.7)
- added REF**: NPTH, NPTH, F.Cu at (83.8, 53.7)
- added REF**: NPTH, NPTH, F.Cu at (82.8, 53.7)
- added REF**: NPTH, NPTH, F.Cu at (81.8, 53.7)
- added REF**: NPTH, NPTH, F.Cu at (80.8, 53.7)
- added REF**: NPTH, NPTH, F.Cu at (92.8, 117.0)
- added REF**: NPTH, NPTH, F.Cu at (79.8, 53.7)
- added REF**: NPTH, NPTH, F.Cu at (74.0, 53.7)
- added REF**: NPTH, NPTH, F.Cu at (73.0, 53.7)
- added REF**: NPTH, NPTH, F.Cu at (72.0, 53.7)
- added REF**: NPTH, NPTH, F.Cu at (71.0, 53.7)
- added REF**: NPTH, NPTH, F.Cu at (70.0, 53.7)
- added REF**: NPTH, NPTH, F.Cu at (69.0, 53.7)
- added REF**: NPTH, NPTH, F.Cu at (63.3, 53.7)
- added REF**: NPTH, NPTH, F.Cu at (62.3, 53.7)
- added REF**: NPTH, NPTH, F.Cu at (61.3, 53.7)
- added REF**: NPTH, NPTH, F.Cu at (92.8, 116.0)
- added REF**: NPTH, NPTH, F.Cu at (60.3, 53.7)
- added REF**: NPTH, NPTH, F.Cu at (59.3, 53.7)
- added REF**: NPTH, NPTH, F.Cu at (58.3, 53.7)
- added REF**: NPTH, NPTH, F.Cu at (46.5, 159.0)
- added REF**: NPTH, NPTH, F.Cu at (96.5, 44.0)
- added REF**: NPTH, NPTH, F.Cu at (46.5, 44.0)
- added REF**: Fiducial, Fiducial, B.Cu at (51.5, 159.0)
- added REF**: Fiducial, Fiducial, F.Cu at (51.5, 159.0)
- added REF**: Fiducial, Fiducial, B.Cu at (91.5, 44.0)
- added REF**: Fiducial, Fiducial, F.Cu at (91.5, 44.0)
- added REF**: NPTH, NPTH, F.Cu at (92.8, 115.0)
- added REF**: Fiducial, Fiducial, B.Cu at (51.5, 44.0)
- added REF**: Fiducial, Fiducial, F.Cu at (51.5, 44.0)
- added REF**: NPTH, NPTH, F.Cu at (92.8, 114.0)
- added REF**: NPTH, NPTH, F.Cu at (92.8, 113.0)
- added REF**: NPTH, NPTH, F.Cu at (50.2, 138.0)
- added REF**: NPTH, NPTH, F.Cu at (92.8, 142.0)
- added REF**: NPTH, NPTH, F.Cu at (50.2, 139.0)
- added REF**: NPTH, NPTH, F.Cu at (50.2, 140.0)
- added REF**: NPTH, NPTH, F.Cu at (50.2, 141.0)
- added REF**: NPTH, NPTH, F.Cu at (50.2, 142.0)
- added REF**: NPTH, NPTH, F.Cu at (50.2, 143.0)
- added REF**: NPTH, NPTH, F.Cu at (50.2, 125.5)
- added REF**: NPTH, NPTH, F.Cu at (50.2, 126.5)
- added REF**: NPTH, NPTH, F.Cu at (50.2, 127.5)
- added REF**: NPTH, NPTH, F.Cu at (50.2, 128.5)
- added REF**: NPTH, NPTH, F.Cu at (50.2, 129.5)
- added REF**: NPTH, NPTH, F.Cu at (92.8, 141.0)
- added REF**: NPTH, NPTH, F.Cu at (50.2, 130.5)
- added REF**: NPTH, NPTH, F.Cu at (50.2, 113.0)
- added REF**: NPTH, NPTH, F.Cu at (50.2, 114.0)
- added REF**: NPTH, NPTH, F.Cu at (50.2, 115.0)
- added REF**: NPTH, NPTH, F.Cu at (50.2, 116.0)
- added REF**: NPTH, NPTH, F.Cu at (50.2, 117.0)
- added REF**: NPTH, NPTH, F.Cu at (50.2, 118.0)
- added REF**: NPTH, NPTH, F.Cu at (92.8, 90.0)
- added REF**: NPTH, NPTH, F.Cu at (92.8, 89.0)
- added REF**: NPTH, NPTH, F.Cu at (92.8, 88.0)
- added REF**: NPTH, NPTH, F.Cu at (92.8, 140.0)
- added REF**: NPTH, NPTH, F.Cu at (92.8, 87.0)
- added REF**: NPTH, NPTH, F.Cu at (92.8, 86.0)
- added REF**: NPTH, NPTH, F.Cu at (92.8, 85.0)
- added REF**: NPTH, NPTH, F.Cu at (92.8, 77.5)
- added REF**: NPTH, NPTH, F.Cu at (92.8, 76.5)
- added REF**: NPTH, NPTH, F.Cu at (92.8, 75.5)
- added REF**: NPTH, NPTH, F.Cu at (92.8, 74.5)
- added REF**: NPTH, NPTH, F.Cu at (92.8, 73.5)
- added REF**: NPTH, NPTH, F.Cu at (92.8, 72.5)
- added REF**: NPTH, NPTH, F.Cu at (92.8, 65.0)
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Connections:
- SW1 pad MP: (no net) -> Board_2-Board_1-GND
- SW1 pad MP: (no net) -> Board_1-Board_1-GND
- SW2 pad MP: (no net) -> Board_2-Board_1-GND
- SW2 pad MP: (no net) -> Board_1-Board_1-GND
- U1 pad 10: Board_2-Board_1-Net-(U1-Pad10) -> (no net)
- U1 pad 11: Board_2-Board_1-Net-(U1-Pad10) -> (no net)
- U1 pad 14: Board_2-Board_1-Net-(U1-Pad10) -> (no net)
- U1 pad 9: Board_2-Board_1-Net-(U1-Pad10) -> (no net)
- U1 pad 10: Board_1-Board_1-Net-(U1-Pad10) -> (no net)
- U1 pad 11: Board_1-Board_1-Net-(U1-Pad10) -> (no net)
- U1 pad 14: Board_1-Board_1-Net-(U1-Pad10) -> (no net)
- U1 pad 9: Board_1-Board_1-Net-(U1-Pad10) -> (no net)
Routing:
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- added copper zone on B.Cu, net Board_1-Board_1-GND
- added copper zone on F.Cu, net Board_1-Board_1-GND
- added copper zone on B.Cu, net Board_2-Board_1-GND
- added copper zone on F.Cu, net Board_2-Board_1-GND
Other:
- outline, holes or cut-outs redrawn
- net class USB_D: clearance 0.1524 -> 0.254
- net class VCC: trace_width 0.2 -> 0.1524
- net class VIN: clearance 0.254 -> 0.1524; trace_width 0.4 -> 0.1524
- board text added: "IO0/~BOOT"
- board text added: "JLCJLCJLCJLC"
- board text added: "neg2led.github.io/esp-pmsa"
- board text added: "v1.0"
- board text removed: "Boot"

Commit message: Deploying to gh-pages from @ neg2led/esp-pmsa@f8f0e89e197d9d7cec6abac82e6cbc78cb6912ec 🚀
Parts:
- removed the C4 at (70.8, 94.5)
- removed the H4 at (52.5, 97.5)
- removed the J2 at (87.5, 60.1)
- removed the REF** at (51.5, 159.0) (x2)
- removed the REF** at (91.5, 44.0) (x2)
- removed the REF** at (51.5, 44.0) (x2)
- removed the U4 at (64.8, 78.5)
- added REF**: Fiducial, Fiducial, B.Cu at (51.5, 159.0)
- added REF**: Fiducial, Fiducial, F.Cu at (51.5, 159.0)
- added REF**: Fiducial, Fiducial, B.Cu at (91.5, 44.0)
- added REF**: Fiducial, Fiducial, F.Cu at (91.5, 44.0)
- added REF**: Fiducial, Fiducial, B.Cu at (51.5, 44.0)
- added REF**: Fiducial, Fiducial, F.Cu at (51.5, 44.0)
- added REF**: NPTH, NPTH, F.Cu at (92.8, 61.0)
- added REF**: NPTH, NPTH, F.Cu at (50.2, 72.5)
- added REF**: NPTH, NPTH, F.Cu at (73.0, 146.4)
- added REF**: NPTH, NPTH, F.Cu at (59.3, 146.0)
- C4: renamed from REF**; value NPTH -> 0.1u; footprint NPTH -> Capacitor_SMD:C_0402_1005Metric
- H4: renamed from REF**; value NPTH -> MP; footprint NPTH -> MountingHole:MountingHole_2.2mm_M2_DIN965_Pad_TopBottom
- J2: renamed from REF**; value NPTH -> ESP-PROG; footprint NPTH -> 11-My-Edits:TC2030_IDCBox_2x03_P1.25mm_Vertical_3D
- U4: renamed from REF**; value NPTH -> XC6210B332MR; footprint NPTH -> Package_TO_SOT_SMD:SOT-23-5
- moved C4 52.0 mm to (70.8, 94.5), turned to 45 degrees
- moved H4 49.0 mm to (52.5, 97.5)
- moved U4 15.7 mm to (64.8, 78.5), turned to 90 degrees
- moved J2 5.34 mm to (87.5, 60.1), turned to 270 degrees

Commit message: Deploying to gh-pages from @ neg2led/esp-pmsa@53209a84ec166707ba2d67fc5a12d877258f9ac0 🚀
Parts:
- removed the C2 at (62.3, 130.5)
- removed the C4 at (70.8, 147.5)
- removed the C4 at (70.8, 94.5)
- removed the C7 at (58.3, 139.9)
- removed the C8 at (58.3, 141.4)
- removed the C8 at (58.3, 88.4)
- removed the R4 at (89.0, 144.7)
- removed the REF** at (92.8, 143.0)
- removed the REF** at (92.8, 127.5)
- removed the REF** at (79.8, 106.8)
- removed the REF** at (74.0, 106.8)
- removed the REF** at (73.0, 106.8)
- removed the REF** at (72.0, 106.8)
- removed the REF** at (71.0, 106.8)
- removed the REF** at (70.0, 106.8)
- removed the REF** at (69.0, 106.8)
- removed the REF** at (63.3, 106.8)
- removed the REF** at (62.3, 106.8)
- removed the REF** at (61.3, 106.8)
- removed the REF** at (92.8, 126.5)
- removed the REF** at (60.3, 106.8)
- removed the REF** at (59.3, 106.8)
- removed the REF** at (58.3, 106.8)
- removed the REF** at (92.8, 125.5)
- removed the REF** at (92.8, 118.0)
- removed the REF** at (92.8, 117.0)
- removed the REF** at (92.8, 116.0)
- removed the REF** at (46.5, 159.0)
- removed the REF** at (46.5, 44.0)
- removed the REF** at (51.5, 159.0) (x2)
- removed the REF** at (91.5, 44.0) (x2)
- removed the REF** at (92.8, 115.0)
- removed the REF** at (51.5, 44.0) (x2)
- removed the REF** at (92.8, 114.0)
- removed the REF** at (92.8, 113.0)
- removed the REF** at (50.2, 138.0)
- removed the REF** at (92.8, 142.0)
- removed the REF** at (50.2, 139.0)
- removed the REF** at (50.2, 140.0)
- removed the REF** at (50.2, 141.0)
- removed the REF** at (50.2, 142.0)
- removed the REF** at (50.2, 143.0)
- removed the REF** at (50.2, 125.5)
- removed the REF** at (50.2, 126.5)
- removed the REF** at (50.2, 127.5)
- removed the REF** at (50.2, 128.5)
- removed the REF** at (50.2, 129.5)
- removed the REF** at (92.8, 141.0)
- removed the REF** at (50.2, 130.5)
- removed the REF** at (50.2, 113.0)
- removed the REF** at (50.2, 114.0)
- removed the REF** at (50.2, 115.0)
- removed the REF** at (50.2, 116.0)
- removed the REF** at (50.2, 117.0)
- removed the REF** at (50.2, 118.0)
- removed the REF** at (92.8, 140.0)
- removed the REF** at (92.8, 139.0)
- removed the REF** at (92.8, 138.0)
- removed the REF** at (92.8, 130.5)
- removed the REF** at (79.8, 146.0)
- removed the REF** at (80.8, 146.0)
- removed the REF** at (81.8, 146.0)
- removed the REF** at (82.8, 146.0)
- removed the REF** at (83.8, 146.0)
- removed the REF** at (84.8, 146.0)
- removed the REF** at (68.9, 152.1)
- removed the REF** at (92.8, 129.5)
- removed the REF** at (69.5, 151.3)
- removed the REF** at (69.6, 150.3)
- removed the REF** at (70.1, 149.3)
- removed the REF** at (70.8, 148.6)
- removed the REF** at (71.5, 147.9)
- removed the REF** at (72.2, 147.1)
- removed the REF** at (73.0, 146.4)
- removed the REF** at (74.0, 146.1)
- removed the REF** at (58.3, 146.0)
- removed the REF** at (59.3, 146.0)
- removed the REF** at (92.8, 128.5)
- removed the REF** at (60.3, 146.0)
- removed the REF** at (61.2, 146.3)
- removed the REF** at (62.0, 146.9)
- removed the REF** at (62.7, 147.6)
- removed the REF** at (63.4, 148.3)
- removed the REF** at (84.8, 106.8)
- removed the REF** at (83.8, 106.8)
- removed the REF** at (82.8, 106.8)
- removed the REF** at (81.8, 106.8)
- removed the REF** at (80.8, 106.8)
- added C4: 0.1u, Capacitor_SMD:C_0402_1005Metric, F.Cu at (118.5, 91.0)
- added C4: 0.1u, Capacitor_SMD:C_0402_1005Metric, F.Cu at (72.5, 91.0)
- added C8: 10u, Capacitor_SMD:C_0603_1608Metric_Pad1.05x0.95mm_HandSolder, F.Cu at (104.3, 88.4)
- added H3: MP, MountingHole:MountingHole_2.2mm_M2_DIN965_Pad_TopBottom, F.Cu at (136.5, 52.5)
- added REF**: NPTH, NPTH, F.Cu at (138.8, 90.0)
- added REF**: NPTH, NPTH, F.Cu at (138.8, 74.5)
- added REF**: NPTH, NPTH, F.Cu at (125.8, 53.7)
- added REF**: NPTH, NPTH, F.Cu at (120.0, 53.7)
- added REF**: NPTH, NPTH, F.Cu at (119.0, 53.7)
- added REF**: NPTH, NPTH, F.Cu at (118.0, 53.7)
- added REF**: NPTH, NPTH, F.Cu at (117.0, 53.7)
- added REF**: NPTH, NPTH, F.Cu at (116.0, 53.7)
- added REF**: NPTH, NPTH, F.Cu at (115.0, 53.7)
- added REF**: NPTH, NPTH, F.Cu at (109.3, 53.7)
- added REF**: NPTH, NPTH, F.Cu at (108.3, 53.7)
- added REF**: NPTH, NPTH, F.Cu at (107.3, 53.7)
- added REF**: NPTH, NPTH, F.Cu at (138.8, 73.5)
- added REF**: NPTH, NPTH, F.Cu at (106.3, 53.7)
- added REF**: NPTH, NPTH, F.Cu at (105.3, 53.7)
- added REF**: NPTH, NPTH, F.Cu at (104.3, 53.7)
- added REF**: NPTH, NPTH, F.Cu at (138.8, 72.5)
- added REF**: NPTH, NPTH, F.Cu at (70.1, 96.3)
- added REF**: NPTH, NPTH, F.Cu at (138.8, 65.0)
- added REF**: NPTH, NPTH, F.Cu at (138.8, 64.0)
- added REF**: NPTH, NPTH, F.Cu at (69.0, 53.7)
- added REF**: NPTH, NPTH, F.Cu at (138.8, 63.0)
- added REF**: NPTH, NPTH, F.Cu at (49.5, 102.5)
- added REF**: NPTH, NPTH, F.Cu at (139.5, 47.5)
- added REF**: NPTH, NPTH, F.Cu at (49.5, 47.5)
- added REF**: Fiducial, Fiducial, B.Cu at (54.5, 102.5)
- added REF**: Fiducial, Fiducial, F.Cu at (54.5, 102.5)
- added REF**: Fiducial, Fiducial, B.Cu at (134.5, 47.5)
- added REF**: Fiducial, Fiducial, F.Cu at (134.5, 47.5)
- added REF**: NPTH, NPTH, F.Cu at (138.8, 62.0)
- added REF**: Fiducial, Fiducial, B.Cu at (54.5, 47.5)
- added REF**: Fiducial, Fiducial, F.Cu at (54.5, 47.5)
- added REF**: NPTH, NPTH, F.Cu at (138.8, 61.0)
- added REF**: NPTH, NPTH, F.Cu at (138.8, 60.0)
- added REF**: NPTH, NPTH, F.Cu at (96.3, 85.0)
- added REF**: NPTH, NPTH, F.Cu at (138.8, 89.0)
- added REF**: NPTH, NPTH, F.Cu at (96.3, 86.0)
- added REF**: NPTH, NPTH, F.Cu at (96.3, 87.0)
- added REF**: NPTH, NPTH, F.Cu at (96.3, 88.0)
- added REF**: NPTH, NPTH, F.Cu at (96.3, 89.0)
- added REF**: NPTH, NPTH, F.Cu at (96.3, 90.0)
- added REF**: NPTH, NPTH, F.Cu at (96.3, 72.5)
- added REF**: NPTH, NPTH, F.Cu at (96.3, 73.5)
- added REF**: NPTH, NPTH, F.Cu at (96.3, 74.5)
- added REF**: NPTH, NPTH, F.Cu at (96.3, 75.5)
- added REF**: NPTH, NPTH, F.Cu at (96.3, 76.5)
- added REF**: NPTH, NPTH, F.Cu at (138.8, 88.0)
- added REF**: NPTH, NPTH, F.Cu at (96.3, 77.5)
- added REF**: NPTH, NPTH, F.Cu at (96.3, 60.0)
- added REF**: NPTH, NPTH, F.Cu at (96.3, 61.0)
- added REF**: NPTH, NPTH, F.Cu at (96.3, 62.0)
- added REF**: NPTH, NPTH, F.Cu at (96.3, 63.0)
- added REF**: NPTH, NPTH, F.Cu at (96.3, 64.0)
- added REF**: NPTH, NPTH, F.Cu at (96.3, 65.0)
- added REF**: NPTH, NPTH, F.Cu at (138.8, 87.0)
- added REF**: NPTH, NPTH, F.Cu at (138.8, 86.0)
- added REF**: NPTH, NPTH, F.Cu at (138.8, 85.0)
- added REF**: NPTH, NPTH, F.Cu at (138.8, 77.5)
- added REF**: NPTH, NPTH, F.Cu at (125.8, 93.0)
- added REF**: NPTH, NPTH, F.Cu at (126.8, 93.0)
- added REF**: NPTH, NPTH, F.Cu at (127.8, 93.0)
- added REF**: NPTH, NPTH, F.Cu at (128.8, 93.0)
- added REF**: NPTH, NPTH, F.Cu at (129.8, 93.0)
- added REF**: NPTH, NPTH, F.Cu at (130.8, 93.0)
- added REF**: NPTH, NPTH, F.Cu at (114.9, 99.1)
- added REF**: NPTH, NPTH, F.Cu at (138.8, 76.5)
- added REF**: NPTH, NPTH, F.Cu at (115.5, 98.3)
- added REF**: NPTH, NPTH, F.Cu at (115.6, 97.3)
- added REF**: NPTH, NPTH, F.Cu at (116.1, 96.3)
- added REF**: NPTH, NPTH, F.Cu at (116.8, 95.6)
- added REF**: NPTH, NPTH, F.Cu at (117.5, 94.9)
- added REF**: NPTH, NPTH, F.Cu at (118.2, 94.1)
- added REF**: NPTH, NPTH, F.Cu at (119.0, 93.4)
- added REF**: NPTH, NPTH, F.Cu at (120.0, 93.1)
- added REF**: NPTH, NPTH, F.Cu at (104.3, 93.0)
- added REF**: NPTH, NPTH, F.Cu at (105.3, 93.0)
- added REF**: NPTH, NPTH, F.Cu at (138.8, 75.5)
- added REF**: NPTH, NPTH, F.Cu at (106.3, 93.0)
- added REF**: NPTH, NPTH, F.Cu at (107.2, 93.3)
- added REF**: NPTH, NPTH, F.Cu at (108.0, 93.9)
- added REF**: NPTH, NPTH, F.Cu at (108.7, 94.6)
- added REF**: NPTH, NPTH, F.Cu at (109.4, 95.3)
- added REF**: NPTH, NPTH, F.Cu at (130.8, 53.7)
- added REF**: NPTH, NPTH, F.Cu at (129.8, 53.7)
- added REF**: NPTH, NPTH, F.Cu at (128.8, 53.7)
- added REF**: NPTH, NPTH, F.Cu at (127.8, 53.7)
- added REF**: NPTH, NPTH, F.Cu at (126.8, 53.7)
- C2: renamed from REF**; value NPTH -> 10u; footprint NPTH -> Capacitor_SMD:C_0402_1005Metric
- C7: renamed from REF**; value NPTH -> 10u; footprint NPTH -> Capacitor_SMD:C_0603_1608Metric_Pad1.05x0.95mm_HandSolder
- C8: renamed from H3; value MP -> 10u; footprint MountingHole:MountingHole_2.2mm_M2_DIN965_Pad_TopBottom -> Capacitor_SMD:C_0603_1608Metric_Pad1.05x0.95mm_HandSolder
- R4: renamed from REF**; value NPTH -> 5k1; footprint NPTH -> Resistor_SMD:R_0402_1005Metric
- moved R3 70.2 mm to (135.0, 92.8)
- moved C1 70.2 mm to (108.3, 79.5)
- moved C3 70.2 mm to (121.0, 76.5)
- moved C5 70.2 mm to (118.0, 76.5)
- moved C9 70.2 mm to (106.5, 62.5)
- moved D1 70.2 mm to (133.5, 72.5)
- moved H1 70.2 mm to (98.5, 52.5)
- moved H2 70.2 mm to (136.5, 97.5)
- moved H4 70.2 mm to (98.5, 97.5)
- moved J1 70.2 mm to (126.0, 88.1)
- moved J2 70.2 mm to (133.5, 60.1)
- moved LOGO1 70.2 mm to (127.5, 78.5)
- moved M1 70.2 mm to (117.5, 72.5)
- moved R1 70.2 mm to (106.5, 70.5)
- moved R2 70.2 mm to (106.5, 68.5)
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Connections:
- C8 pad 1: Board_2-Board_1-GND -> Board_1-Board_1-+5V
Routing:
- net Board_2-Board_1-/VCC_ALS: track 20.5 -> 19.8 mm
- net Board_1-Board_1-/VCC_ALS: track 20.5 -> 19.8 mm
Other:
- board size 60 x 120 mm -> 100 x 60 mm

Commit message: Deploying to gh-pages from @ neg2led/esp-pmsa@5792303937cde9c3b92ca60e7ea9c0f6023d491c 🚀
Parts:
- removed the REF** at (54.5, 102.5) (x2)
- removed the REF** at (134.5, 47.5) (x2)
- removed the REF** at (54.5, 47.5) (x2)
- added REF**: Fiducial, Fiducial, B.Cu at (54.5, 102.5)
- added REF**: Fiducial, Fiducial, F.Cu at (54.5, 102.5)
- added REF**: Fiducial, Fiducial, B.Cu at (134.5, 47.5)
- added REF**: Fiducial, Fiducial, F.Cu at (134.5, 47.5)
- added REF**: Fiducial, Fiducial, B.Cu at (54.5, 47.5)
- added REF**: Fiducial, Fiducial, F.Cu at (54.5, 47.5)
Routing:
- net Board_2-Board_1-/VCC_BME: track 30.0 -> 31.0 mm
- net Board_1-Board_1-/VCC_BME: track 30.0 -> 31.0 mm
Changed lines of the file:
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@@
     (thickness 1.6002)
     (drawings 3088)
-    (tracks 526)
+    (tracks 528)
     (zones 0)
     (modules 217)
@@
   (segment (start 69.301001 96.201001) (end 69.301001 95.701001) (width 0.1524) (layer F.Cu) (net 13))
   (segment (start 68.438501 96.601001) (end 68.901001 96.601001) (width 0.1524) (layer F.Cu) (net 13))
+  (segment (start 72.501001 92.501001) (end 72.501001 91.481001) (width 0.127) (layer F.Cu) (net 13))
   (via (at 89.551001 66.501001) (size 0.6) (drill 0.3) (layers F.Cu B.Cu) (net 14))
   (via (at 89.551001 81.151001) (size 0.6) (drill 0.3) (layers F.Cu B.Cu) (net 14))
@@
   (segment (start 115.303317 96.201001) (end 115.303317 95.701001) (width 0.1524) (layer F.Cu) (net 34))
   (segment (start 114.440817 96.601001) (end 114.903317 96.601001) (width 0.1524) (layer F.Cu) (net 34))
+  (segment (start 118.503317 92.501001) (end 118.503317 91.481001) (width 0.127) (layer F.Cu) (net 34))
   (via (at 135.553317 66.501001) (size 0.6) (drill 0.3) (layers F.Cu B.Cu) (net 35))
   (via (at 135.553317 81.151001) (size 0.6) (drill 0.3) (layers F.Cu B.Cu) (net 35))
