File: boards/esp-pmsa.kicad_pcb (KiCad board)
At the start: 2 copper layers, 40 x 47.5 mm, 12 parts, among them M1 PMSA003, U1 WeMos_D1_mini_Labels, U2 BME68x, U3 OPT3001DNPT

Commit message: Deploying to gh-pages from @ neg2led/esp-pmsa@a730e507301c682fc7d8a88894b304163d40722a 🚀
Parts:
- removed the C7 at (133.2, 109.8)
- added C3: 1uF, Capacitor_SMD:C_0402_1005Metric, F.Cu at (149.2, 119.0)
- C7: renamed from C3; value 1uF -> 10uF; footprint Capacitor_SMD:C_0402_1005Metric -> Capacitor_SMD:C_0603_1608Metric_Pad1.05x0.95mm_HandSolder
- moved C7 18.5 mm to (133.2, 109.8), turned to 180 degrees
Connections:
- C7 pad 1: Board_1-/VCC_SENS -> Board_1-+5V

Commit message: Deploying to gh-pages from @ neg2led/esp-pmsa@060c7214fca1917f5e98065bfc5be80db49c411f 🚀
Parts:
- removed the M1 at (150.0, 97.5)
- added H2: MP, MountingHole:MountingHole_2.2mm_M2_DIN965_Pad_TopBottom, F.Cu at (167.5, 120.0)
- M1: renamed from H2; value MP -> PMSA003; footprint MountingHole:MountingHole_2.2mm_M2_DIN965_Pad_TopBottom -> 12-Collected-Footprints:PMSA003; moved to B.Cu
- moved M1 28.5 mm to (150.0, 97.5)
Connections:
- M1 pad 1: Board_1-GND -> Board_1-+5V
