File: boards/esp-pmsa.kicad_pcb (KiCad board)
At the start: 2 copper layers, 40 x 47.5 mm, 12 parts, among them M1 PMSA003, U1 WeMos_D1_mini_Labels, U2 BME68x, U3 OPT3001DNPT

Commit message: Deploying to gh-pages from @ neg2led/esp-pmsa@e03a36f01e21f29b520752c6169685313d9a0f2f 🚀
Parts:
- added C1: 10u, Capacitor_SMD:C_0402_1005Metric, F.Cu at (146.6, 103.9)
- added C2: 10u, Capacitor_SMD:C_0402_1005Metric, F.Cu at (141.9, 103.1)
- added C5: 1u, Capacitor_SMD:C_0402_1005Metric, F.Cu at (150.5, 101.5)
- added C6: 0.1u, Capacitor_SMD:C_0402_1005Metric, F.Cu at (142.5, 115.2)
- added C9: 0.1u, Capacitor_SMD:C_0402_1005Metric, F.Cu at (138.0, 87.0)
- added D1: APA104-12-3535, 21-SnapEDA-zip:LED_APA104-12-3535, F.Cu at (166.0, 97.5)
- added J1: USB_C_Receptacle_USB2.0_304S-ACP16, 41-EasyEDA-Edits:USB-C-SMD_TYPEC-304S-ACP16, F.Cu at (158.5, 113.0)
- added J2: ESP-PROG, 11-My-Edits:TC2030_IDCBox_2x03_P1.25mm_Vertical_3D, F.Cu at (166.0, 85.0)
- added R1: 4k7, Resistor_SMD:R_0402_1005Metric, F.Cu at (137.5, 95.2)
- added R2: 4k7, Resistor_SMD:R_0402_1005Metric, F.Cu at (137.5, 93.8)
- added R3: 5k1, Resistor_SMD:R_0402_1005Metric, F.Cu at (167.5, 117.8)
- added R4: 5k1, Resistor_SMD:R_0402_1005Metric, F.Cu at (167.5, 116.7)
- added SW1: Reset, 41-EasyEDA-Edits:SW-SMD_SKSLLAE010-3D, F.Cu at (130.4, 107.0)
- added SW2: Boot, 41-EasyEDA-Edits:SW-SMD_SKSLLAE010-3D, F.Cu at (169.6, 107.0)
- added U4: XC6220B331MR, Package_TO_SOT_SMD:SOT-23-5, F.Cu at (144.2, 103.5)
- C3: value 1uF -> 1u
- C4: value 100nF -> 0.1u
- C7, C8: value 10uF -> 10u
- U1: value WeMos_D1_mini_Labels -> ESP32-C3F; footprint 11-My-Edits:WEMOS_D1_mini -> 11-My-Edits:ESP-12H
- moved U3 35.3 mm to (145.7, 122.1), turned to 0 degrees
- moved C3 18.0 mm to (153.5, 101.5), turned to 0 degrees
- moved U1 9.00 mm to (150.0, 87.0)
- moved C8 6.25 mm to (136.8, 113.4), turned to 0 degrees
- moved U2 5.00 mm to (145.8, 122.1)
- moved C4 4.14 mm to (149.0, 115.2), turned to 180 degrees
- moved C7 4.13 mm to (136.8, 111.9), turned to 0 degrees
- moved H2 2.92 mm to (169.0, 122.5)
- moved H4 2.92 mm to (131.0, 122.5)
- moved H1 1.50 mm to (131.0, 77.5)
- moved H3 1.50 mm to (169.0, 77.5)
Connections:
- C3 pad 1: Board_1-/VCC_SENS -> Board_1-/VCC_BME
- C4 pad 1: Board_1-GND -> Board_1-/VCC_BME
- C4 pad 2: Board_1-/VCC_SENS -> Board_1-GND
- M1 pad 8: Board_1-Net-(M1-Pad8) -> Board_1-Net-(M1-Pad6)
- U1 pad 1: Board_1-/~WAKE -> Board_1-/PMS_RX
- U1 pad 10: Board_1-GND -> Board_1-Net-(U1-Pad10)
- U1 pad 11: Board_1-Net-(U1-Pad11) -> Board_1-Net-(U1-Pad10)
- U1 pad 12: Board_1-/VCC_SENS -> Board_1-/VCC_ALS
- U1 pad 13: Board_1-/SDA -> Board_1-/VCC_BME
- U1 pad 14: Board_1-/SCL -> Board_1-Net-(U1-Pad10)
- U1 pad 15: Board_1-/U0RXD -> Board_1-GND
- U1 pad 16: Board_1-/U0TXD -> (no net)
- U1 pad 2: Board_1-Net-(U1-Pad2) -> Board_1-/PMS_TX
- U1 pad 3: Board_1-/~WAKE -> Board_1-/~RST
- U1 pad 4: Board_1-/~PMS_RST -> Board_1-/~PMS_SET
- U1 pad 5: Board_1-/~PMS_SET -> Board_1-/~PMS_RST
- U1 pad 6: Board_1-/PMS_TX -> Board_1-/SDA
- U1 pad 7: Board_1-/PMS_RX -> Board_1-/SCL
- U1 pad 9: Board_1-+5V -> Board_1-Net-(U1-Pad10)
- U2 pad 2: Board_1-/VCC_SENS -> Board_1-/VCC_BME
- U2 pad 6: Board_1-/VCC_SENS -> Board_1-/VCC_BME
- U2 pad 8: Board_1-/VCC_SENS -> Board_1-/VCC_BME
- U3 pad 1: Board_1-/VCC_SENS -> Board_1-/VCC_ALS
- U3 pad 5: Board_1-Net-(U3-Pad5) -> (no net)
Routing:
- net Board_1-/~RST: track 0.00 -> 53.6 mm, vias 0 -> 3
- net Board_1-/VCC_SENS: track 42.8 -> 0.00 mm, vias 1 -> 0
- net Board_1-/SCL: track 35.5 -> 0.00 mm
- net Board_1-+5V: track 39.4 -> 5.03 mm
- net Board_1-/SDA: track 33.8 -> 0.00 mm
- net Board_1-/~BOOT: track 0.00 -> 32.2 mm, vias 0 -> 2
- net Board_1-/PMS_RX: track 17.0 -> 34.1 mm
- net Board_1-Net-(J1-PadA5): track 0.00 -> 16.2 mm
- net Board_1-/PMS_TX: track 13.5 -> 29.6 mm, vias 0 -> 1
- net Board_1-Net-(J1-PadB5): track 0.00 -> 13.1 mm
- net Board_1-/~PMS_SET: track 14.8 -> 25.0 mm, vias 0 -> 1
- net Board_1-/U0TXD: track 0.00 -> 8.41 mm
- net Board_1-/U0RXD: track 0.00 -> 8.10 mm
- net Board_1-/~WAKE: track 7.79 -> 0.00 mm
- net Board_1-/~PMS_RST: track 23.1 -> 29.6 mm, vias 0 -> 1
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- removed copper zone on B.Cu, net Board_1-GND
- removed copper zone on F.Cu, net Board_1-GND
Other:
- board size 40 x 47.5 mm -> 43 x 50 mm
- board text added: "Boot"
- board text added: "Reset"
- board text removed: "vriska did nothing wrong"

Commit message: Deploying to gh-pages from @ neg2led/esp-pmsa@1a288ce33808fbc405a6c24b3a385c7c225d67b1 🚀
Parts:
- added LOGO1: neggles logo, 10-My-Footprints:neggle-logo-0.12, F.Cu at (160.0, 103.5)
- U2: moved to F.Cu
- U4: value XC6220B331MR -> XC6210B332MR
- moved U3 8.63 mm to (145.8, 113.5), turned to 180 degrees
- moved C1 5.86 mm to (140.8, 104.5)
- moved C6 5.71 mm to (148.0, 113.7), turned to 90 degrees
- moved C4 4.26 mm to (149.2, 119.5), turned to 45 degrees
- moved R1 1.56 mm to (139.0, 95.5)
- moved R2 1.56 mm to (139.0, 93.5)
- moved C2 1.24 mm to (140.8, 102.5)
- moved C9 1.11 mm to (139.0, 87.5), turned to 0 degrees
- moved U4 1.00 mm to (143.2, 103.5)
- moved U2 0.12 mm to (145.8, 122.0)
Connections:
- SW1 pad MP: (no net) -> Board_1-GND
- SW2 pad MP: (no net) -> Board_1-GND
- U1 pad 10: Board_1-Net-(U1-Pad10) -> (no net)
- U1 pad 11: Board_1-Net-(U1-Pad10) -> (no net)
- U1 pad 14: Board_1-Net-(U1-Pad10) -> (no net)
- U1 pad 9: Board_1-Net-(U1-Pad10) -> (no net)
Routing:
- net Board_1-+5V: track 5.03 -> 55.6 mm
- net Board_1-/SDA: track 0.00 -> 41.0 mm, vias 0 -> 3
- net Board_1-/SCL: track 0.00 -> 38.0 mm, vias 0 -> 2
- net Board_1-/USB_D-: track 0.00 -> 29.4 mm, vias 0 -> 2
- net Board_1-/USB_D+: track 0.00 -> 27.7 mm, vias 0 -> 2
- net Board_1-/VCC_BME: track 4.63 -> 30.0 mm, vias 0 -> 2
- net Board_1-/VCC_ALS: track 0.00 -> 20.5 mm, vias 0 -> 2
- net Board_1-+3V3: track 0.00 -> 14.5 mm
- net Board_1-/RGB: track 0.00 -> 7.94 mm
- net Board_1-GND: track 0.00 -> 3.52 mm, vias 7 -> 58
- net Board_1-/~RST: track 53.6 -> 51.8 mm
- added copper zone on B.Cu, net Board_1-GND
- added copper zone on F.Cu, net Board_1-GND
Other:
- net class USB_D: clearance 0.1524 -> 0.254
- net class VCC: trace_width 0.2 -> 0.1524
- net class VIN: clearance 0.254 -> 0.1524; trace_width 0.4 -> 0.1524
- board text added: "IO0/~BOOT"
- board text added: "JLCJLCJLCJLC"
- board text added: "neg2led.github.io/esp-pmsa"
- board text added: "v1.0"
- board text removed: "Boot"

Commit message: Deploying to gh-pages from @ neg2led/esp-pmsa@53209a84ec166707ba2d67fc5a12d877258f9ac0 🚀
Parts:
- moved C4 3.91 mm to (151.0, 116.0), turned to 90 degrees
Routing:
- net Board_1-/VCC_ALS: track 20.5 -> 19.8 mm
Changed lines of the file:
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@@
     (thickness 1.6002)
     (drawings 419)
-    (tracks 264)
+    (tracks 263)
     (zones 0)
     (modules 28)
@@
     (solder_mask_min_width 0.12)
     (aux_axis_origin 0 0)
-    (grid_origin 171.5 78.5)
     (visible_elements 7FFFFFFF)
     (pcbplotparams
@@
   )
   (module Capacitor_SMD:C_0402_1005Metric (layer F.Cu)
-    (at 149.25 119.5 45)
+    (at 151 116 90)
     (descr "Capacitor SMD 0402 (1005 Metric), square (rectangular) end terminal, IPC_7351 nominal, (Body size source: IPC-SM-782 page 76, https://www.pcb-3d.com/wordpress/wp-content/uploads/ipc-sm-782a_amendment_1_and_2.pdf), generated with kicad-footprint-generator")
     (tags capacitor)
     (attr smd)
-    (fp_text reference C4 (at 1.891511 -0.22981 unlocked) (layer F.SilkS)
+    (fp_text reference C4 (at 1.6 0 unlocked) (layer F.SilkS)
       (effects (font (size 0.75 0.75) (thickness 0.12)))
     )
-    (fp_text value 0.1u (at -1.1 0 315) (layer F.Fab)
+    (fp_text value 0.1u (at -1.1 0 180) (layer F.Fab)
       (effects (font (size 0.25 0.25) (thickness 0.05)))
     )
@@
     (fp_line (start -0.5 -0.25) (end 0.5 -0.25) (layer F.Fab) (width 0.1))
     (fp_line (start -0.5 0.25) (end -0.5 -0.25) (layer F.Fab) (width 0.1))
-    (pad 1 smd roundrect (at -0.48 0 45) (size 0.56 0.62) (layers F.Cu F.Paste F.Mask) (roundrect_rratio 0.25)
+    (pad 1 smd roundrect (at -0.48 0 90) (size 0.56 0.62) (layers F.Cu F.Paste F.Mask) (roundrect_rratio 0.25)
       (net 13 Board_1-/VCC_BME))
-    (pad 2 smd roundrect (at 0.48 0 45) (size 0.56 0.62) (layers F.Cu F.Paste F.Mask) (roundrect_rratio 0.25)
+    (pad 2 smd roundrect (at 0.48 0 90) (size 0.56 0.62) (layers F.Cu F.Paste F.Mask) (roundrect_rratio 0.25)
       (net 18 Board_1-GND))
     (model ${KISYS3DMOD}/Capacitor_SMD.3dshapes/C_0402_1005Metric.wrl
@@
   (segment (start 147.97 114.15) (end 148 114.18) (width 0.1524) (layer F.Cu) (net 12))
   (segment (start 146.65 114.15) (end 147.97 114.15) (width 0.1524) (layer F.Cu) (net 12))
-  (segment (start 151.5 114.15) (end 151.5 114.15) (width 0.1524) (layer B.Cu) (net 12))
-  (via (at 151.5 114.15) (size 0.6) (drill 0.3) (layers F.Cu B.Cu) (net 12))
+  (via (at 151 113.5) (size 0.6) (drill 0.3) (layers F.Cu B.Cu) (net 12))
   (segment (start 151.85 103.35) (end 151 102.5) (width 0.1524) (layer B.Cu) (net 12))
-  (segment (start 151.85 113.8) (end 151.85 103.35) (width 0.1524) (layer B.Cu) (net 12))
-  (segment (start 151.5 114.15) (end 151.85 113.8) (width 0.1524) (layer B.Cu) (net 12))
-  (segment (start 148.03 114.15) (end 151.5 114.15) (width 0.1524) (layer F.Cu) (net 12))
+  (segment (start 151.85 112.65) (end 151.85 103.35) (width 0.1524) (layer B.Cu) (net 12))
+  (segment (start 151 113.5) (end 151.85 112.65) (width 0.1524) (layer B.Cu) (net 12))
+  (segment (start 150.35 114.15) (end 151 113.5) (width 0.1524) (layer F.Cu) (net 12))
+  (segment (start 148.03 114.15) (end 150.35 114.15) (width 0.1524) (layer F.Cu) (net 12))
   (segment (start 148 114.18) (end 148.03 114.15) (width 0.1524) (layer F.Cu) (net 12))
   (segment (start 146.15 121.6) (end 145.35 122.4) (width 0.127) (layer F.Cu) (net 13))
@@
   (segment (start 153 102.5) (end 153 101.5) (width 0.1524) (layer F.Cu) (net 13))
   (segment (start 153 101.5) (end 153 99) (width 0.1524) (layer F.Cu) (net 13))
-  (segment (start 148.910589 120.089411) (end 148.910589 119.839411) (width 0.1524) (layer F.Cu) (net 13))
-  (segment (start 147.4 121.6) (end 148.910589 120.089411) (width 0.1524) (layer F.Cu) (net 13))
+  (via (at 151 117.5) (size 0.6) (drill 0.3) (layers F.Cu B.Cu) (net 13))
+  (segment (start 153 102.5) (end 152.15 103.35) (width 0.1524) (layer B.Cu) (net 13))
+  (segment (start 152.15 103.35) (end 152.15 116.35) (width 0.1524) (layer B.Cu) (net 13))
+  (segment (start 152.15 116.35) (end 151 117.5) (width 0.1524) (layer B.Cu) (net 13))
+  (segment (start 147.8 120.7) (end 151 117.5) (width 0.1524) (layer F.Cu) (net 13))
+  (segment (start 147.4 121.6) (end 147.8 121.2) (width 0.1524) (layer F.Cu) (net 13))
+  (segment (start 147.8 121.2) (end 147.8 120.7) (width 0.1524) (layer F.Cu) (net 13))
   (segment (start 146.9375 121.6) (end 147.4 121.6) (width 0.1524) (layer F.Cu) (net 13))
-  (via (at 151.5 116.3) (size 0.6) (drill 0.3) (layers F.Cu B.Cu) (net 13))
-  (segment (start 152.15 115.65) (end 151.5 116.3) (width 0.1524) (layer B.Cu) (net 13))
-  (segment (start 152.15 103.35) (end 152.15 115.65) (width 0.1524) (layer B.Cu) (net 13))
-  (segment (start 153 102.5) (end 152.15 103.35) (width 0.1524) (layer B.Cu) (net 13))
-  (segment (start 148.910589 119.839411) (end 148.910589 118.889411) (width 0.1524) (layer F.Cu) (net 13))
-  (segment (start 148.910589 118.889411) (end 151.5 116.3) (width 0.1524) (layer F.Cu) (net 13))
   (via (at 168.05 91.5) (size 0.6) (drill 0.3) (layers F.Cu B.Cu) (net 14))
   (via (at 168.05 106.15) (size 0.6) (drill 0.3) (layers F.Cu B.Cu) (net 14))
@@
   (via (at 166 96.625) (size 0.6) (drill 0.3) (layers F.Cu B.Cu) (net 18))
   (segment (start 167.75 96.625) (end 166 96.625) (width 0.127) (layer F.Cu) (net 18))
-  (via (at 150.5 118.55) (size 0.6) (drill 0.3) (layers F.Cu B.Cu) (net 18))
   (via (at 155 97.5) (size 0.6) (drill 0.3) (layers F.Cu B.Cu) (net 18))
   (via (at 135 98.5) (size 0.6) (drill 0.3) (layers F.Cu B.Cu) (net 18))
@@
   (via (at 160 103.5) (size 0.6) (drill 0.3) (layers F.Cu B.Cu) (net 18))
   (via (at 165 108.5) (size 0.6) (drill 0.3) (layers F.Cu B.Cu) (net 18))
-  (via (at 150 108.5) (size 0.6) (drill 0.3) (layers F.Cu B.Cu) (net 18))
-  (via (at 150 113.5) (size 0.6) (drill 0.3) (layers F.Cu B.Cu) (net 18))
+  (via (at 148.5 110) (size 0.6) (drill 0.3) (layers F.Cu B.Cu) (net 18))
   (via (at 155 93.5) (size 0.6) (drill 0.3) (layers F.Cu B.Cu) (net 18))
   (via (at 155 88.5) (size 0.6) (drill 0.3) (layers F.Cu B.Cu) (net 18))
@@
   (via (at 170 118.5) (size 0.6) (drill 0.3) (layers F.Cu B.Cu) (net 18))
   (segment (start 145.75 112.65) (end 145.75 114.425) (width 0.508) (layer F.Cu) (net 18))
+  (via (at 148.5 105) (size 0.6) (drill 0.3) (layers F.Cu B.Cu) (net 18))
+  (via (at 153.5 105) (size 0.6) (drill 0.3) (layers F.Cu B.Cu) (net 18))
   (segment (start 166.59 117.4) (end 166.99 117.8) (width 0.127) (layer F.Cu) (net 19))
   (segment (start 158.25 117.4) (end 166.59 117.4) (width 0.127) (layer F.Cu) (net 19))

Commit message: Deploying to gh-pages from @ neg2led/esp-pmsa@5792303937cde9c3b92ca60e7ea9c0f6023d491c 🚀
Routing:
- net Board_1-/VCC_BME: track 30.0 -> 31.0 mm
Changed lines of the file:
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@@
     (thickness 1.6002)
     (drawings 419)
-    (tracks 263)
+    (tracks 264)
     (zones 0)
     (modules 28)
@@
   (segment (start 147.8 121.2) (end 147.8 120.7) (width 0.1524) (layer F.Cu) (net 13))
   (segment (start 146.9375 121.6) (end 147.4 121.6) (width 0.1524) (layer F.Cu) (net 13))
+  (segment (start 151 117.5) (end 151 116.48) (width 0.127) (layer F.Cu) (net 13))
   (via (at 168.05 91.5) (size 0.6) (drill 0.3) (layers F.Cu B.Cu) (net 14))
   (via (at 168.05 106.15) (size 0.6) (drill 0.3) (layers F.Cu B.Cu) (net 14))
